File: CDH/CDH-v4.1.brd (EAGLE design)
At the start: 90.6 x 91.8 mm, 47 parts

Commit message: Updates to CDH subsystem
Changes to be committed:
	deleted:    CDH-v3.7.pro
	deleted:    CDH-v3.7_PCB_Final_Design.pdf
	renamed:    CDH-v3.7.brd -> CDH-v4.1.brd
	new file:   CDH-v4.1.pro
	renamed:    CDH-v3.7.sch -> CDH-v4.1.sch
Parts:
- moved H1 5.06 mm to (42.3, 82.7)
- moved H2 5.06 mm to (42.3, 87.8)
Connections:
- removed net PC_Q6_RS232: H2.21, U$1.44
- removed net Q6_PC_RS232: H2.25, U$1.42
- new net N$18: U$1.42
- new net N$19: U$1.44
- net +3V3: now also H2.36, H2.38; no longer H1.36, H1.38
- net ANTENNA_DEPLOYMENT_+V: now also H1.1; no longer H2.1
- net ANTENNA_DEPLOYMENT_GND: now also H1.3; no longer H2.3
- net BATTERY_HEATER_+V: now also H1.4; no longer H2.4
- net BATTERY_HEATER_-V: now also H1.6; no longer H2.6
- net BATTERY_THRMSTOR2_+V: now also H1.12; no longer H2.12
- net BATTERY_THRMSTOR_+V: now also H1.8; no longer H2.8
- net BATTERY_THRMSTOR_-V: now also H1.10; no longer H2.10
- net BOTTOM_TEMP_SOLAR_PANEL-1: now also H2.9; no longer H1.9
- net BOTTOM_TEMP_SOLAR_PANEL-2: now also H2.11; no longer H1.11
- net BOTTOM_TEMP_SOLAR_PANEL-3: now also H2.13; no longer H1.13
- net BOTTOM_TEMP_SOLAR_PANEL-4: now also H2.15; no longer H1.15
- net ELEC_BAY_TEMP_1: now also H2.50; no longer H1.50
- net EXTERNAL_POWER_+V: now also H2.52; no longer H1.51
- net EXTERNAL_POWER_GND: now also H2.51; no longer H1.52
- net GND: now also H1.15, H1.23, H1.27, H1.34, H1.37, H1.41, H1.44, H1.45, H1.48, H1.49, H1.52, H2.16, H2.17, H2.22, H2.26, H2.4, U$6.1, U$6.10, U$6.11, U$6.12, U$6.13, U$6.14, U$6.19, U$6.2, U$6.7, U$6.8, U$6.9; no longer H1.16, H1.17, H1.22, H1.26, H1.4, H2.15, H2.23, H2.27, H2.34, H2.37, H2.41, H2.44, H2.45, H2.48, H2.49, H2.52
- net MECH_DEPLOY_SWITCH_+V: now also H2.31; no longer H1.31
- net MECH_DEPLOY_SWITCH_-V: now also H2.33; no longer H1.33
- net N$1: now also H2.6; no longer H1.6
- net N$11: now also H2.2; no longer H1.2
- net N$13: now also H2.49; no longer H1.49
- net N$15: now also H2.47; no longer H1.47
- net N$22: now also H2.34; no longer H1.34
- net N$27: now also H2.44; no longer H1.44
- net N$4: now also H2.8; no longer H1.8
- net N$5: now also H2.48; no longer H1.48
- net N$6: now also H2.10; no longer H1.10
- net N$78: now also H2.39; no longer H1.39
- net N$79: now also H2.41; no longer H1.41
- net N$80: now also H2.43; no longer H1.43
- net N$81: now also H2.40; no longer H1.40
- net N$83: now also H1.46; no longer H2.46
- net N$84: now also H1.50; no longer H2.50
- net N$9: now also H2.12; no longer H1.12
- net PA3_PC_RS232: now also H1.25
- net PC_PA3_RS232: now also H1.21
- net POW_3V3: now also H1.16, H1.20; no longer H2.16, H2.20
- net POW_5V: now also H1.26, H1.28; no longer H2.26, H2.28
- net POW_9V: now also H1.22, H1.24; no longer H2.22, H2.24
- net POW_BATT_GND: now also H1.33; no longer H2.33
- net POW_BATT_VOUT: now also H1.35; no longer H2.35
- net POW_RADIO_3.3V: now also H2.27; no longer H1.27
- net POW_RADIO_3.3VSYS: now also H2.28; no longer H1.28
- net POW_RADIO_GND: now also H2.29, H2.30, H2.32; no longer H1.29, H1.30, H1.32
- net POW_RADIO_VBATT: now also H2.45, H2.46; no longer H1.45, H1.46
- net Q6_AIN_0: now also H1.39; no longer H2.39
- net Q6_AIN_1: now also H1.43; no longer H2.43
- net Q6_AOUT_0: now also H1.47; no longer H2.47
- net Q6_AOUT_1: now also H1.51; no longer H2.51
- net Q6_GPIO_0: now also H1.13; no longer H2.13
- net Q6_GPIO_10: now also H1.32; no longer H2.32
- net Q6_GPIO_13: now also H1.36; no longer H2.36
- net Q6_GPIO_14: now also H1.38; no longer H2.38
- net Q6_GPIO_15: now also H1.40; no longer H2.40
- net Q6_GPIO_2: now also H2.24; no longer H1.24
- net Q6_GPIO_6: now also H1.7; no longer H2.7
- net Q6_GPIO_7: now also H1.9; no longer H2.9
- net Q6_GPIO_8: now also H1.11; no longer H2.11
- net Q6_I2C_SCL_1: now also H2.20; no longer H1.20
- net Q6_I2C_SDA_1: now also H2.18; no longer H1.18
- net Q6_RADIO_UART_RX: now also H1.18; no longer H2.18
- net Q6_RADIO_UART_TX: now also H1.17; no longer H2.17
- net Q6_SPI_CS0: now also H2.37; no longer H1.37
- net Q6_SPI_CS1: now also H2.25; no longer H1.25
- net Q6_SPI_SCLK: now also H2.21; no longer H1.21
- net Q6_SPI_SDI_MISO: now also H2.35; no longer H1.35
- net Q6_SPI_SDO_MOSI: now also H2.23; no longer H1.23
- net SLR_PNL_GND: now also H1.30; no longer H2.30
- net SOLAR_PANEL_1_3: now also H1.29; no longer H2.29
- net SOLAR_PANEL_2_4: now also H1.2; no longer H2.2
- net SOLAR_PANEL_GND: now also H1.31; no longer H2.31
- net THERMALGND1: now also H1.5; no longer H2.5
- net TOP_TEMP_SOLAR_PANEL-1: now also H2.1; no longer H1.1
- net TOP_TEMP_SOLAR_PANEL-2: now also H2.3; no longer H1.3
- net TOP_TEMP_SOLAR_PANEL-3: now also H2.5; no longer H1.5
- net TOP_TEMP_SOLAR_PANEL-4: now also H2.7; no longer H1.7
Routing:
- net PC_PA3_RS232: track 0.00 -> 91.6 mm, vias 0 -> 6
- net PC_Q6_RS232: track 76.4 -> 0.00 mm, vias 3 -> 0
- net Q6_PC_RS232: track 68.5 -> 0.00 mm, vias 4 -> 0
- net GND: track 453.1 -> 487.1 mm
- net EXTERNAL_POWER_+V: track 18.2 -> 20.5 mm
- net EXTERNAL_POWER_GND: track 25.3 -> 23.8 mm
Other:
- board text added: "1"
- board text added: "10"
- board text added: "2"
- board text added: "3"
- board text added: "4"
- board text added: "49"
- board text added: "5"
- board text added: "50"
- board text added: "51"
- board text added: "52"
- board text added: "6"
- board text added: "7"
- board text added: "8"
- board text added: "9"
