File: Payload External/payload-externalPCB-version2-modif2.brd (EAGLE design)
At the start: 94.8 x 83 mm, 78 parts

Commit message: Added working version of v2 payload external schematic Added Libraries dir
Changes to be committed:
	new file:   Libraries/space-concordia-power.lbr
	modified:   Payload External/payload-externalPCB-version2-modif2.brd
	modified:   Payload External/payload-externalPCB-version2-modif2.sch
Parts:
- removed C17, C27, C28, C29: (no value), rcl:C1812
- added C36, C37: 1 uF, rcl:C2220K
- C1: value (none) -> 10 uF
- C10, C11, C12, C19, C20, C21, C22, C23, C24, C3, C30, C31, C32, C33, C34, C35, C4, C5, C6, C7: value (none) -> 100 uF
- C13, C14, C25, C26: value (none) -> 0.01 uF
- C15, C16: value (none) -> 2.2 uF; device rcl:C1812 -> rcl:C2220K
- C18: value (none) -> 15 pF
- C2: value (none) -> 0.033 uF
- R1, R12: value (none) -> 4.75 MOhm
- R10: value (none) -> 43.1 kOhm
- R11, R17, R7: value (none) -> 4.87 kOhm
- R18, R6: value (none) -> 47 kOhm
- R19: value (none) -> 1.2 MOhm
- R2: value (none) -> 10 Ohm
- R20: value (none) -> 4.85 kOhm
- R3: value (none) -> 179 Ohm
- R4: value (none) -> 1MOhm
- R5: value (none) -> 4 MOhm
- R8: value (none) -> 100 kOhm
- R9: value (none) -> 102 kOhm
- moved C16 45.5 mm to (-83.5, 44.1), turned to 0 degrees
- moved R7 19.3 mm to (-46.3, 34.4), turned to 180 degrees
- moved C33 7.66 mm to (-89.5, 10.4), turned to 270 degrees
- moved C15 5.86 mm to (-46.2, 16.8), turned to 0 degrees
- moved C21 5.85 mm to (-38.2, 32.3)
- moved C35 5.71 mm to (-89.4, 23.6), turned to 180 degrees
- moved C11 5.66 mm to (-46.4, 45.2)
- moved C7 5.44 mm to (-38.3, 41.9)
- moved C30 5.39 mm to (-94.4, 10.5), turned to 270 degrees
- moved C6 5.21 mm to (-38.2, 37.0), turned to 180 degrees
- moved C19 5.02 mm to (-38.2, 22.5)
- moved C20 4.97 mm to (-38.2, 27.2), turned to 180 degrees
- moved C4 4.60 mm to (-34.4, 17.5), turned to 270 degrees
- moved C5 4.05 mm to (-39.0, 17.5), turned to 270 degrees
- moved C34 3.98 mm to (-90.1, 18.1), turned to 180 degrees
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Connections:
- removed net N$10: C4.2, C5.1
- removed net N$13: C19.2, C20.1
- removed net N$14: C20.2, C21.1
- removed net N$15: C19.1, C5.2
- removed net N$16: C6.2, C7.1
- removed net N$18: C12.1, C7.2
- removed net N$19: C21.2, C6.1
- removed net N$20: C11.1, C12.2
- removed net N$21: C15.2, C16.1
- removed net N$22: C16.2, C17.1
- removed net N$29: C10.1, U$10.6
- removed net N$30: C10.2, C22.1
- removed net N$31: C22.2, C23.1
- removed net N$32: C30.2, C31.1
- removed net N$33: C31.2, C32.1
- removed net N$34: C23.2, C30.1
- removed net N$35: C33.2, C34.1
- removed net N$36: C34.2, C35.1
- removed net N$37: C32.2, C33.1
- removed net N$38: C24.1, C35.2
- removed net N$39: C27.2, C28.1
- removed net N$40: C28.2, C29.1
- net GND2: now also C10.2, C12.2, C15.2, C16.2, C19.2, C20.2, C21.2, C22.2, C23.2, C3.2, C30.2, C31.2, C32.2, C33.2, C34.2, C35.2, C36.2, C37.2, C4.2, C5.2, C6.2, C7.2; no longer C17.2, C29.2
- net HV_G-M-ANODE1: now also C36.1
- net HV_G-M-ANODE2: now also C16.1, C37.1; no longer C27.1
- net N$6: now also C11.1, C12.1, C19.1, C20.1, C21.1, C4.1, C5.1, C6.1, C7.1
- net N$9: now also C10.1, C22.1, C23.1, C24.1, C30.1, C31.1, C32.1, C33.1, C34.1, C35.1, U$10.6; no longer C3.2, C4.1
Routing:
- net GND2: track 225.3 -> 351.5 mm, vias 7 -> 9
- net N$9: track 3.66 -> 54.7 mm
- net N$6: track 5.76 -> 52.0 mm
- net HV_G-M-ANODE1: track 103.4 -> 115.4 mm
- net N$29: track 10.7 -> 0.00 mm
- net HV_G-M-ANODE2: track 87.0 -> 97.5 mm
- net N$40: track 8.13 -> 0.00 mm
- net N$14: track 8.09 -> 0.00 mm
- net N$15: track 7.94 -> 0.00 mm
- net N$16: track 7.70 -> 0.00 mm
- net N$18: track 6.56 -> 0.00 mm
- net N$37: track 6.56 -> 0.00 mm
- net GND1: track 106.8 -> 113.2 mm
- net N$35: track 6.26 -> 0.00 mm
- net N$39: track 5.98 -> 0.00 mm
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