File: Payload External/payload-externalPCB-version2-modif2.sch (EAGLE design)
At the start: 47 parts

Commit message: Further updates to CDH Added design v2 of the payload external pcb
Changes to be committed:
	deleted:    CDH/CDH-v4.1.brd
	deleted:    CDH/CDH-v4.1.pro
	new file:   CDH/CDH-v4.11-A-DS1338-tcc-test-redesign.brd
	renamed:    CDH/CDH-v4.1.sch -> CDH/CDH-v4.11-A-DS1338-tcc-test-redesign.sch

	new file:   Payload External/payload-externalPCB-version2-modif2.brd
	new file:   Payload External/payload-externalPCB-version2-modif2.sch
Parts:
- removed ADC_TEMP_1, ADC_TEMP_2: AD7998-1, analog-devices:AD7998-1
- removed D1: BB141, diode:BB141
- removed H1, H2: ESQ-125-XX-X-D, ESQ-126-XX-X-D:ESQ-125-XX-X-D
- added C20, C21, C22, C23, C24, C30, C31, C32, C33, C34, C35: (no value), rcl:C-EUC1210
- added C25, C26: (no value), rcl:C-EUC1206
- added C27, C28, C29: (no value), rcl:C-USC1812
- added R18: (no value), rcl:R-US_R1210
- added R19: (no value), rcl:R-US_R1206
- added R20: (no value), rcl:R-US_R2010
- added U$10: PM61300-4-RC, Payload-board:PM61300-4-RC
- added U$11, U$12, U$7, U$8: S1J-SCHEMATICS, Payload-board:S1J-SCHEMATICS
- added U$13, U$14: RESISTOR-J-LEAD-5W, Payload-board:RESISTOR-J-LEAD-5W
- added U$15, U$16, U$23: PZT3904-SOT223-SCHEMATICS, Payload-board:PZT3904-SOT223-SCHEMATICS
- added U$17, U$18, U$19, U$20, U$21, U$22: SMBJ5388B-ZENER-DIODE-200V, Payload-board:SMBJ5388B-ZENER-DIODE-200V
- added U$9: IRLIZ14GPBF-ND-SCHEMATICS, Payload-board:IRLIZ14GPBF-ND-SCHEMATICS
- C1, C12, C3, C4, C5, C6, C7, C8: value 1uF -> (none); device rcl:C-EUC2012 -> rcl:C-EUC1210
- C10, C11: value 0.1uF -> (none); device rcl:C-EUC2012 -> rcl:C-EUC1210
- C13: value 1uF -> (none); device rcl:C-EUC2012 -> rcl:C-EUC1206
- C14: value 0.1uF -> (none); device rcl:C-EUC2012 -> rcl:C-EUC1206
- C15: value 10uF -> (none); device rcl:C-EUC2012 -> rcl:C-USC1812
- C16: value 1uF -> (none); device rcl:C-EUC2012 -> rcl:C-USC1812
- C17: value 0.1uF -> (none); device rcl:C-EUC2012 -> rcl:C-USC1812
- C18, C2: value 1uF -> (none); device rcl:C-EUC2012 -> rcl:C-USC0805
- C19: value 10uF -> (none); device rcl:C-EUC2012 -> rcl:C-EUC1210
- C9: value 10uF -> (none); device rcl:C-EUC2012 -> rcl:C-USC0805
- R1, R12, R9: value 220k -> (none); device resistor:R-US_R2012 -> rcl:R-US_R1206
- R10: value THERMISTOR-2,5 -> (none); device varistor:THERMISTOR-2,5 -> rcl:R-US_R2010
- R11: value 100k -> (none); device resistor:R-US_R2012 -> rcl:R-US_R1210
- R13, R14, R15, R2, R3, R4, R5, R7, R8: value 220k -> (none); device resistor:R-US_R2012 -> rcl:R-US_R2010
- R16, R17: value 10k -> (none); device resistor:R-US_R2012 -> rcl:R-US_R2010
- R6: value 220k -> (none); device resistor:R-US_R2012 -> rcl:R-US_R1210
- U$1: value SMFC -> M80-5000000M2-04-331-00-000; device SFMC-125-02-S-D:SMFC -> Payload-board:M80-5000000M2-04-331-00-000
- U$2: value M80-5000000M1-10-331-000 -> M80-8670805; device harwin:M80-5000000M1-10-331-000 -> Payload-board:M80-8670805
- U$3: value M80-5000000M1-10-331-00-000 -> M80-8670805; device harwin:M80-5000000M1-10-331-00-000 -> Payload-board:M80-8670805
- U$4: value ADM6316/ADM6320 -> IRLIZ14GPBF-ND-SCHEMATICS; device analog-devices:ADM6316/ADM6320 -> Payload-board:IRLIZ14GPBF-ND-SCHEMATICS
- U$5: value (none) -> PM61300-4-RC; device adafruit:CR1220SMT -> Payload-board:PM61300-4-RC
- U$6: value DS3232 -> PZT3904-SOT223-SCHEMATICS; device maxim:DS3232 -> Payload-board:PZT3904-SOT223-SCHEMATICS
Connections:
- removed net +3V3: ADC_TEMP_1.VDD, ADC_TEMP_1.VDD1, ADC_TEMP_1.~CONVST, ADC_TEMP_2.VDD, ADC_TEMP_2.VDD1, ADC_TEMP_2.~CONVST, C10.1, C11.1, C14.1, C15.1, C17.1, C9.1, H2.36, H2.38, R1.2, R12.2, R13.2, R14.2, R15.2, R16.1, R17.2, R2.2, R3.2, R4.2, R5.2, R6.2, R7.2, R8.2, U$1.C32, U$4.VCC, U$6.VCC
- removed net ANTENNA_DEPLOYMENT_+V: H1.1
- removed net ANTENNA_DEPLOYMENT_GND: H1.3
- removed net BATTERY_HEATER_+V: H1.4, U$2.X6
- removed net BATTERY_HEATER_-V: H1.6, U$2.X7
- removed net BATTERY_THRMSTOR2_+V: H1.12, U$2.X10
- removed net BATTERY_THRMSTOR_+V: H1.8, U$2.X8
- removed net BATTERY_THRMSTOR_-V: H1.10, U$2.X9
- removed net BATT_TEMP_0: ADC_TEMP_2.VIN4, C16.2, R13.1
- removed net BATT_TEMP_1: ADC_TEMP_2.VIN3, C18.2, R12.1, U$2.X3
- removed net BOTTOM_TEMP_SOLAR_PANEL-1: ADC_TEMP_1.VIN5, C4.2, H2.9, R5.1
- removed net BOTTOM_TEMP_SOLAR_PANEL-2: ADC_TEMP_1.VIN6, C3.2, H2.11, R6.1
- removed net BOTTOM_TEMP_SOLAR_PANEL-3: ADC_TEMP_1.VIN7, C2.2, H2.13, R7.1
- removed net BOTTOM_TEMP_SOLAR_PANEL-4: ADC_TEMP_1.VIN8, C1.2, H2.15, R8.1
- removed net ELEC_BAY_TEMP_0: ADC_TEMP_2.VIN8, C12.2, R10.1, R15.1
- removed net ELEC_BAY_TEMP_1: ADC_TEMP_2.VIN7, C13.2, H2.50, R14.1
- removed net EXTERNAL_POWER_+V: H2.52, U$3.X4
- removed net EXTERNAL_POWER_GND: H2.51, U$3.X3
- removed net GND: ADC_TEMP_1.AS, C1.1, C10.2, C11.2, C12.1, C13.1, C14.2, C15.2, C16.1, C17.2, C18.1, C19.1, C2.1, C3.1, C4.1, C5.1, C6.1, C7.1, C8.1, C9.2, D1.A, H1.15, H1.19, H1.23, H1.27, H1.34, H1.37, H1.41, H1.44, H1.45, H1.48, H1.49, H1.52, H2.16, H2.17, H2.19, H2.22, H2.26, H2.4, R11.2, R9.2, U$1.C1, U$1.C10, U$1.C2, U$1.C27, U$1.C28, U$1.C39, U$1.C40, U$1.C47, U$1.C48, U$1.C7, U$1.C8, U$1.C9, U$4.GND, U$5.-, U$6.GND, U$6.N.C.1, U$6.N.C.10, U$6.N.C.11, U$6.N.C.2, U$6.N.C.3, U$6.N.C.4, U$6.N.C.5, U$6.N.C.6, U$6.N.C.7, U$6.N.C.8, U$6.N.C.9
- removed net MECH_DEPLOY_SWITCH_+V: H2.31, U$2.X4
- removed net MECH_DEPLOY_SWITCH_-V: H2.33, U$2.X5
- removed net N$17: H2.14
- removed net N$654643543: H1.14
- removed net N$78: H2.39
- removed net N$79: H2.41
- removed net N$80: H2.43
- removed net N$81: H2.40
- removed net N$82: H2.42
- removed net N$83: H1.46
- removed net N$84: H1.50
- removed net PA3_GPIO_6: U$1.C35
- removed net PA3_GPIO_7: U$1.C37
- removed net PA3_GPIO_8: U$1.C36
- removed net PA3_GPIO_9: U$1.C38
- removed net PA3_JTAG_TCK: U$1.C29
- removed net PA3_JTAG_TDI: U$1.C33
- removed net PA3_JTAG_TDO: U$1.C30
- removed net PA3_JTAG_TMS: U$1.C31
- removed net PA3_PC_RS232: H1.25, U$1.C41
- removed net PC_PA3_RS232: H1.21, U$1.C43
- removed net POW_3V3: H1.16, H1.20
- removed net POW_5V: H1.26, H1.28, U$1.C49, U$1.C50
- removed net POW_9V: H1.22, H1.24
- removed net POW_BATT_GND: H1.33, U$3.X1
- removed net POW_BATT_VOUT: H1.35, U$3.X2
- removed net POW_RADIO_3.3V: H2.27
- removed net POW_RADIO_3.3VSYS: H2.28
- removed net POW_RADIO_GND: H2.29, H2.30, H2.32
- removed net POW_RADIO_VBATT: H2.45, H2.46
- removed net PWR_CTRL: R11.1, U$1.C45, U$4.~RESET
- removed net Q6_AIN_0: H1.39, U$1.C3
- removed net Q6_AIN_1: H1.43, U$1.C5
- removed net Q6_AOUT_0: H1.47, U$1.C4
- removed net Q6_AOUT_1: H1.51, U$1.C6
- removed net Q6_GPIO_0: H1.13, U$1.C11, U$4.WDI
- removed net Q6_GPIO_10: H1.32, U$1.C16
- removed net Q6_GPIO_13: H1.36, U$1.C22
- removed net Q6_GPIO_14: H1.38, U$1.C24
- removed net Q6_GPIO_15: H1.40, U$1.C26
- removed net Q6_GPIO_2: H2.24, U$1.C15
- removed net Q6_GPIO_6: H1.7, U$1.C23
- removed net Q6_GPIO_7: H1.9, U$1.C25
- removed net Q6_GPIO_8: H1.11, U$1.C12
- removed net Q6_I2C_SCL_1: ADC_TEMP_1.SCL, ADC_TEMP_2.SCL, H2.20, U$1.C13, U$6.SCL
- removed net Q6_I2C_SDA_1: ADC_TEMP_1.SDA, ADC_TEMP_2.SDA, H2.18, U$1.C14, U$6.SDA
- removed net Q6_RADIO_UART_RX: H1.18
- removed net Q6_RADIO_UART_TX: H1.17
- removed net Q6_SPI_CS0: H2.37, U$1.C20
- removed net Q6_SPI_CS1: H2.25, U$1.C21
- removed net Q6_SPI_SCLK: H2.21, U$1.C17
- removed net Q6_SPI_SDI_MISO: H2.35, U$1.C19
- removed net Q6_SPI_SDO_MOSI: H2.23, U$1.C18
- removed net REF_IN: ADC_TEMP_1.REF_IN, ADC_TEMP_2.REF_IN, C19.2, D1.C, R17.1
- removed net SLR_PNL_GND: H1.30
- removed net SOLAR_PANEL_1_3: H1.29
- removed net SOLAR_PANEL_2_4: H1.2
- removed net SOLAR_PANEL_GND: H1.31
- removed net THERMALGND1: ADC_TEMP_1.AGND, ADC_TEMP_1.AGND1, ADC_TEMP_1.AGND2, ADC_TEMP_1.AGND3, ADC_TEMP_2.AGND, ADC_TEMP_2.AGND1, ADC_TEMP_2.AGND2, ADC_TEMP_2.AGND3, H1.5, R10.2, R9.1
- removed net TOP_TEMP_SOLAR_PANEL-1: ADC_TEMP_1.VIN1, C8.2, H2.1, R1.1
- removed net TOP_TEMP_SOLAR_PANEL-2: ADC_TEMP_1.VIN2, C7.2, H2.3, R2.1
- removed net TOP_TEMP_SOLAR_PANEL-3: ADC_TEMP_1.VIN3, C6.2, H2.5, R3.1
- removed net TOP_TEMP_SOLAR_PANEL-4: ADC_TEMP_1.VIN4, C5.2, H2.7, R4.1
- removed net VBAT: U$5.+, U$5.+1, U$6.VBAT
- removed net ~MANUAL_RESET: U$4.~MR
- removed net ~PA3_JAG_TRST: U$1.C34
- removed net ~WAKE_UP: U$1.C46
- new net 5V: R10.2, U$15.C, U$16.C, U$23.C, U$3.P$1
- new net G-M-CATHODE: R19.2, R8.2, U$1.P$2
- new net G-M-COUNTS: R10.1, U$2.P$3, U$6.C
- new net G-M-OUTPUT: U$1.P$3
- new net G-M-OUTPUT-AMPLITUDE: R20.1, U$2.P$8, U$23.E
- new net GND1: C1.2, C8.2, R13.1, R15.1, R17.1, R18.1, R2.1, R20.2, R4.1, R6.1, R7.1, U$3.P$2, U$4.S, U$9.S
- new net GND2: C11.2, C14.2, C17.2, C18.2, C24.2, C26.2, C29.2, R11.1, R16.1, R5.1, R9.1, U$12.A, U$19.P$1, U$22.P$1, U$3.P$3, U$8.A
- new net GND3: U$3.P$4, U$6.E
- new net HV_G-M-ANODE1: C14.1, C15.1, R1.2, R5.2, U$1.P$1, U$17.P$2, U$7.C
- new net HV_G-M-ANODE2: C26.1, C27.1, R12.2, R16.2, U$1.P$4, U$11.C, U$20.P$2
- new net HV_OUTPUT1: R7.2, U$15.E, U$2.P$5
- new net HV_OUTPUT2: R17.2, U$16.E, U$2.P$6
- new net N$10: C4.2, C5.1
- new net N$14: C20.2, C21.1
- new net N$16: C6.2, C7.1
- new net N$20: C11.1, C12.2
- new net N$21: C15.2, C16.1
- new net N$23: R14.1, U$9.G
- new net N$24: C9.2, R13.2
- new net N$25: U$10.3, U$14.P$2
- new net N$26: C9.1, U$14.P$1, U$9.D
- new net N$28: C25.1, U$10.10
- new net N$29: C10.1, U$10.6
- new net N$30: C10.2, C22.1
- new net N$31: C22.2, C23.1
- new net N$32: C30.2, C31.1
- new net N$33: C31.2, C32.1
- new net N$34: C23.2, C30.1
- new net N$35: C33.2, C34.1
- new net N$36: C34.2, C35.1
- new net N$37: C32.2, C33.1
- new net N$38: C24.1, C35.2
- new net N$39: C27.2, C28.1
- new net N$40: C28.2, C29.1
- new net N$41: C25.2, U$11.A, U$12.C
- new net N$42: U$18.P$1, U$19.P$2
- new net N$43: U$20.P$1, U$21.P$2
- new net N$45: U$21.P$1, U$22.P$2
- new net N$46: C18.1, R11.2, R8.1, U$6.B
- new net N$47: R19.1, R9.2, U$23.B
- new net PULSE1: R3.2, R4.2, U$2.P$1
- new net PULSE2: R14.2, R15.2, U$2.P$7
- new net VOLTAGE_SWEEP1: C1.1, U$2.P$2, U$5.1
- new net VOLTAGE_SWEEP2: C8.1, U$10.1, U$2.P$4
- net N$1: now also R3.1, U$4.G; no longer H2.6
- net N$11: now also C2.1, U$13.P$1, U$4.D; no longer H2.2
- net N$13: now also C19.2, C20.1; no longer H2.49
- net N$15: now also C19.1, C5.2; no longer H2.47
- net N$18: now also C12.1, C7.2; no longer U$1.C42
- net N$19: now also C21.2, C6.1; no longer U$1.C44
- net N$2: now also U$17.P$1, U$18.P$2; no longer H1.42
- net N$22: now also C16.2, C17.1; no longer H2.34
- net N$27: now also R1.1, R6.2, U$15.B; no longer H2.44
- net N$3: now also C13.1, U$5.10; no longer ADC_TEMP_2.AS, R16.2
- net N$4: now also C13.2, U$7.A, U$8.C; no longer H2.8
- net N$5: now also R12.1, R18.2, U$16.B; no longer H2.48
- net N$6: now also C3.1, U$5.6; no longer H2.10
- net N$7: now also U$13.P$2, U$5.3; no longer U$6.~RST
- net N$8: now also C2.2, R2.2; no longer U$6.~INT/SQW
- net N$9: now also C3.2, C4.1; no longer H2.12
Other:
- note removed: "15V_CTL"
- note removed: "3V3_CTL"
- note removed: "ANT_CTL"
- note removed: "BATTERY / ELEC BAY / COMMS / PAYLOAD TEMP SENSORS"
- note removed: "BATT_TEMP_0"
- note removed: "BATT_TEMP_1"
- note removed: "COMMS_ATTENA_TEMP"
- note removed: "ELEC_BAY_TEMP_0"
- note removed: "ELEC_BAY_TEMP_1"
- note removed: "PAY_TEMP_0"
- note removed: "PAY_TEMP_1"
- note removed: "POW_RADIO_GND"
- note removed: "Q6-Connector"
- note removed: "Q6_AOUT_0"
- note removed: "Q6_AOUT_1"
- note removed: "Q6_GPIO_10"
- note removed: "SOLAR PANEL TEMP SENSORS"
- note removed: "SOLAR_PANEL_2_4"
- note removed: "WATCH_DOG_INPUT"
- moved on the sheet: C1, C10, C11, C12, C13, C14, C15, C16, C17, C18, C19, C2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

Commit message: Added working version of v2 payload external schematic Added Libraries dir
Changes to be committed:
	new file:   Libraries/space-concordia-power.lbr
	modified:   Payload External/payload-externalPCB-version2-modif2.brd
	modified:   Payload External/payload-externalPCB-version2-modif2.sch
Parts:
- removed C17, C27, C28, C29: (no value), rcl:C-USC1812
- added C36, C37: 1 uF, rcl:C-USC2220K
- C1: value (none) -> 10 uF
- C10, C11, C12, C19, C20, C21, C22, C23, C24, C3, C30, C31, C32, C33, C34, C35, C4, C5, C6, C7: value (none) -> 100 uF
- C13, C14, C25, C26: value (none) -> 0.01 uF
- C15, C16: value (none) -> 2.2 uF; device rcl:C-USC1812 -> rcl:C-USC2220K
- C18: value (none) -> 15 pF
- C2: value (none) -> 0.033 uF
- R1, R12: value (none) -> 4.75 MOhm
- R10: value (none) -> 43.1 kOhm
- R11, R17, R7: value (none) -> 4.87 kOhm
- R18, R6: value (none) -> 47 kOhm
- R19: value (none) -> 1.2 MOhm
- R2: value (none) -> 10 Ohm
- R20: value (none) -> 4.85 kOhm
- R3: value (none) -> 179 Ohm
- R4: value (none) -> 1MOhm
- R5: value (none) -> 4 MOhm
- R8: value (none) -> 100 kOhm
- R9: value (none) -> 102 kOhm
Connections:
- removed net N$10: C4.2, C5.1
- removed net N$13: C19.2, C20.1
- removed net N$14: C20.2, C21.1
- removed net N$15: C19.1, C5.2
- removed net N$16: C6.2, C7.1
- removed net N$18: C12.1, C7.2
- removed net N$19: C21.2, C6.1
- removed net N$20: C11.1, C12.2
- removed net N$21: C15.2, C16.1
- removed net N$22: C16.2, C17.1
- removed net N$29: C10.1, U$10.6
- removed net N$30: C10.2, C22.1
- removed net N$31: C22.2, C23.1
- removed net N$32: C30.2, C31.1
- removed net N$33: C31.2, C32.1
- removed net N$34: C23.2, C30.1
- removed net N$35: C33.2, C34.1
- removed net N$36: C34.2, C35.1
- removed net N$37: C32.2, C33.1
- removed net N$38: C24.1, C35.2
- removed net N$39: C27.2, C28.1
- removed net N$40: C28.2, C29.1
- net GND2: now also C10.2, C12.2, C15.2, C16.2, C19.2, C20.2, C21.2, C22.2, C23.2, C3.2, C30.2, C31.2, C32.2, C33.2, C34.2, C35.2, C36.2, C37.2, C4.2, C5.2, C6.2, C7.2; no longer C17.2, C29.2
- net HV_G-M-ANODE1: now also C36.1
- net HV_G-M-ANODE2: now also C16.1, C37.1; no longer C27.1
- net N$6: now also C11.1, C12.1, C19.1, C20.1, C21.1, C4.1, C5.1, C6.1, C7.1
- net N$9: now also C10.1, C22.1, C23.1, C24.1, C30.1, C31.1, C32.1, C33.1, C34.1, C35.1, U$10.6; no longer C3.2, C4.1
Other:
- moved on the sheet: C10, C11, C12, C15, C16, C19, C20, C21, C22, C23, C24, C3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
