File: Payload Internal - Auxiliary/Payload v2.1.sch (EAGLE design)
At the start: 11 parts

Commit message: Updated Payload internal schem with notes from "20131201 - Continuity Check" Added connections to wiring harness schematic as per "20131201 - Continuity Check"
Other:
- note added: "*Note: This is the "+X" 16pin Conn"
- note added: "*Note: This is the "-X" 16pin Conn"
Changed lines of the file:
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@@
 <?xml version="1.0" encoding="utf-8"?>
 <!DOCTYPE eagle SYSTEM "eagle.dtd">
-<eagle version="6.2">
+<eagle version="7.3.0">
 <drawing>
 <settings>
@@
 <text x="-128.27" y="66.04" size="1.778" layer="95">POW_RADIO_GND</text>
 <text x="-128.27" y="63.5" size="1.778" layer="95">POW_RADIO_GND</text>
+<text x="-287.02" y="106.68" size="1.778" layer="152">*Note: This is the "-X" 16pin Conn</text>
+<text x="-287.02" y="68.58" size="1.778" layer="152">*Note: This is the "+X" 16pin Conn</text>
 </plain>
 <instances>
