File: Payload Internal - Auxiliary/Payload v2.1.sch (EAGLE design)
At the start: 11 parts, among them J30 M80-866XXXX, J31 M80-866XXXX

Commit message: Revert "Fixed all the trivial wiring issues for the CDH, Diplexer, EPS and wiring harness schematics"
This reverts commits
  6713d85a6277b26f983fd7a52d0f95a7f9e4e046.
  086194ae58682b6763f31692a26cd4dac33df983
  82b42737f0fe6cd82dfea4a4ae7507beb01cc7b8

This revert is required because changing/connecting net names in eagle will automatically modify or destroy PCB traces associated with those netnames.
Updating the schematics and PCBs will need to be redone carefully to ensure no traces are destroyed.

	modified:   CDH-V3.7/CDH-v3.7.brd
	modified:   CDH-V3.7/CDH-v3.7.sch
	modified:   Diplexer/diplexer_v4rev0-schematic.sch
	modified:   EPS/eps-v1-0.brd
	modified:   EPS/eps-v1-0.sch
	modified:   Payload Internal - Auxiliary/Payload v2.1.brd
	modified:   Payload Internal - Auxiliary/Payload v2.1.sch
	modified:   Wiring Harness/wiring-harness-complete-v1.0.sch
Connections:
- net BATTERY_THRMSTOR1_+V renamed BATTERY_THRMSTOR_+V
- net BATTERY_THRMSTOR2_+V renamed BATTERY_THERMSTOR_2+
- net POW_9V renamed 9V
- net POW_RADIO_VBATT renamed POW_5V
- net THERMALGND1 renamed THERMALGND
- removed net EXTERNAL_POWER_V+: H2.52
- removed net N$1: H2.6
- removed net N$6: H2.10
- removed net POW_RADIO_3V3: H2.27, H2.28
- new net EXTERNAL_POWER_+V: H2.51
- new net N$19: H2.37
- new net N$89.: H2.21
- new net N$90: H2.23
- new net N$91: H2.25
- net EXTERNAL_POWER_GND: now also H2.52; no longer H2.51
- net N$4: now also H2.35; no longer H2.8
- net POW_RADIO_3.3V: now also H2.27, H2.28
- net Q6_SPI_SCLK: now also H2.6; no longer H2.21
- net Q6_SPI_SDI_MISO: now also H2.10; no longer H2.35
- net Q6_SPI_SDO_MOSI: now also H2.8; no longer H2.23
Other:
- note added: "POW_RADIO_VBATT"
Changed lines of the file:
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@@
 <?xml version="1.0" encoding="utf-8"?>
 <!DOCTYPE eagle SYSTEM "eagle.dtd">
-<eagle version="7.3.0">
+<eagle version="7.2.0">
 <drawing>
 <settings>
@@
 <text x="-129.54" y="22.86" size="1.778" layer="95">SOLAR_PANEL_2_4</text>
 <text x="-111.86" y="-25.01" size="1.778" layer="95">3V3_CTL</text>
+<text x="-195.58" y="66.04" size="1.778" layer="95">POW_RADIO_GND</text>
+<text x="-189.23" y="45.72" size="1.778" layer="95">POW_RADIO_VBATT</text>
+<text x="-124.46" y="45.72" size="1.778" layer="95">POW_RADIO_VBATT</text>
+<text x="-128.27" y="66.04" size="1.778" layer="95">POW_RADIO_GND</text>
+<text x="-128.27" y="63.5" size="1.778" layer="95">POW_RADIO_GND</text>
 </plain>
 <instances>
@@
 </segment>
 </net>
+<net name="N$19" class="0">
+<segment>
+<pinref part="H2" gate="G$1" pin="37"/>
+<wire x1="-162.56" y1="55.88" x2="-205.74" y2="55.88" width="0.1524" layer="91"/>
+<label x="-203.2" y="55.88" size="1.778" layer="95"/>
+</segment>
+</net>
 <net name="N$22" class="0">
 <segment>
@@
 <wire x1="-139.7" y1="60.96" x2="-109.22" y2="60.96" width="0.1524" layer="91"/>
 <label x="-137.16" y="60.96" size="1.778" layer="95"/>
+</segment>
+</net>
+<net name="N$90" class="0">
+<segment>
+<pinref part="H2" gate="G$1" pin="23"/>
+<wire x1="-162.56" y1="73.66" x2="-205.74" y2="73.66" width="0.1524" layer="91"/>
+<label x="-203.2" y="73.66" size="1.778" layer="95"/>
 </segment>
 </net>
@@
 <wire x1="-162.56" y1="-17.78" x2="-190.5" y2="-17.78" width="0.1524" layer="91"/>
 <label x="-187.96" y="-17.78" size="1.778" layer="95"/>
+</segment>
+</net>
+<net name="Q6_SPI_SDO_MOSI" class="0">
+<segment>
+<wire x1="-139.7" y1="93.98" x2="-106.68" y2="93.98" width="0.1524" layer="91"/>
+<pinref part="H2" gate="G$1" pin="8"/>
+<label x="-137.16" y="93.98" size="1.778" layer="95"/>
 </segment>
 </net>
@@
 </segment>
 </net>
-<net name="POW_RADIO_VBATT" class="0">
+<net name="POW_5V" class="0">
 <segment>
 <pinref part="H1" gate="G$1" pin="28"/>
@@
 </segment>
 </net>
+<net name="N$89." class="0">
+<segment>
+<pinref part="H2" gate="G$1" pin="21"/>
+<wire x1="-205.74" y1="76.2" x2="-162.56" y2="76.2" width="0.1524" layer="91"/>
+<label x="-203.2" y="76.2" size="1.778" layer="95"/>
+</segment>
+</net>
+<net name="Q6_SPI_SCLK" class="0">
+<segment>
+<pinref part="H2" gate="G$1" pin="6"/>
+<wire x1="-109.22" y1="96.52" x2="-139.7" y2="96.52" width="0.1524" layer="91"/>
+<label x="-137.16" y="96.52" size="1.778" layer="95"/>
+</segment>
+</net>
+<net name="Q6_SPI_SDI_MISO" class="0">
+<segment>
+<pinref part="H2" gate="G$1" pin="10"/>
+<wire x1="-139.7" y1="91.44" x2="-106.68" y2="91.44" width="0.1524" layer="91"/>
+<label x="-137.16" y="91.44" size="1.778" layer="95"/>
+</segment>
+</net>
 <net name="Q6_AIN_1" class="0">
 <segment>
@@
 </segment>
 </net>
+<net name="N$91" class="0">
+<segment>
+<pinref part="H2" gate="G$1" pin="25"/>
+<wire x1="-204.47" y1="71.12" x2="-162.56" y2="71.12" width="0.1524" layer="91"/>
+<label x="-203.2" y="71.12" size="1.778" layer="95"/>
+</segment>
+</net>
 <net name="POW_RADIO_3.3V" class="0">
+<segment>
+<pinref part="H2" gate="G$1" pin="27"/>
+<wire x1="-162.56" y1="68.58" x2="-205.74" y2="68.58" width="0.1524" layer="91"/>
+<label x="-203.2" y="68.58" size="1.778" layer="95"/>
+</segment>
 <segment>
 <pinref part="H1" gate="G$1" pin="16"/>
@@
 <label x="-129.54" y="5.08" size="1.778" layer="95"/>
 </segment>
+<segment>
+<pinref part="H2" gate="G$1" pin="28"/>
+<wire x1="-139.7" y1="68.58" x2="-106.68" y2="68.58" width="0.1524" layer="91"/>
+<label x="-137.16" y="68.58" size="1.778" layer="95"/>
+</segment>
 </net>
 <net name="POW_3V3" class="0">
@@
 </segment>
 </net>
-<net name="BATTERY_THRMSTOR1_+V" class="0">
+<net name="BATTERY_THRMSTOR_+V" class="0">
 <segment>
 <pinref part="H1" gate="G$1" pin="8"/>
@@
 </segment>
 </net>
-<net name="Q6_SPI_SDI_MISO" class="0">
+<net name="N$4" class="0">
 <segment>
 <pinref part="H2" gate="G$1" pin="35"/>
@@
 </segment>
 </net>
-<net name="EXTERNAL_POWER_V+" class="0">
+<net name="EXTERNAL_POWER_GND" class="0">
 <segment>
 <pinref part="H2" gate="G$1" pin="52"/>
@@
 </segment>
 </net>
-<net name="EXTERNAL_POWER_GND" class="0">
+<net name="EXTERNAL_POWER_+V" class="0">
 <segment>
 <pinref part="H2" gate="G$1" pin="51"/>
@@
 </segment>
 </net>
-<net name="THERMALGND1" class="0">
+<net name="THERMALGND" class="0">
 <segment>
 <pinref part="H1" gate="G$1" pin="5"/>
@@
 </segment>
 </net>
-<net name="POW_9V" class="0">
+<net name="9V" class="0">
 <segment>
 <pinref part="H1" gate="G$1" pin="22"/>
@@
 </segment>
 </net>
-<net name="N$654643543" class="0">
+<net name="N$6546" class="0">
 <segment>
 <pinref part="H1" gate="G$1" pin="14"/>
@@
 </segment>
 </net>
-<net name="BATTERY_THRMSTOR2_+V" class="0">
+<net name="BATTERY_THERMSTOR_2+" class="0">
 <segment>
 <pinref part="H1" gate="G$1" pin="12"/>
@@
 </segment>
 </net>
-<net name="POW_RADIO_3V3" class="0">
-<segment>
-<pinref part="H2" gate="G$1" pin="27"/>
-<wire x1="-162.56" y1="68.58" x2="-205.74" y2="68.58" width="0.1524" layer="91"/>
-<label x="-203.2" y="68.58" size="1.778" layer="95"/>
-</segment>
-<segment>
-<pinref part="H2" gate="G$1" pin="28"/>
-<wire x1="-139.7" y1="68.58" x2="-106.68" y2="68.58" width="0.1524" layer="91"/>
-<label x="-137.16" y="68.58" size="1.778" layer="95"/>
-</segment>
-</net>
-<net name="N$6" class="0">
-<segment>
-<pinref part="H2" gate="G$1" pin="10"/>
-<wire x1="-139.7" y1="91.44" x2="-109.22" y2="91.44" width="0.1524" layer="91"/>
-<label x="-135.89" y="91.44" size="1.778" layer="95"/>
-</segment>
-</net>
-<net name="Q6_SPI_SDO_MOSI" class="0">
-<segment>
-<pinref part="H2" gate="G$1" pin="23"/>
-<wire x1="-162.56" y1="73.66" x2="-205.74" y2="73.66" width="0.1524" layer="91"/>
-<label x="-203.2" y="73.66" size="1.778" layer="95"/>
-</segment>
-</net>
-<net name="N$1" class="0">
-<segment>
-<pinref part="H2" gate="G$1" pin="6"/>
-<wire x1="-139.7" y1="96.52" x2="-109.22" y2="96.52" width="0.1524" layer="91"/>
-<label x="-135.89" y="96.52" size="1.778" layer="95"/>
-</segment>
-</net>
-<net name="N$4" class="0">
-<segment>
-<pinref part="H2" gate="G$1" pin="8"/>
-<wire x1="-139.7" y1="93.98" x2="-109.22" y2="93.98" width="0.1524" layer="91"/>
-<label x="-135.89" y="93.98" size="1.778" layer="95"/>
-</segment>
-</net>
-<net name="Q6_SPI_SCLK" class="0">
-<segment>
-<pinref part="H2" gate="G$1" pin="21"/>
-<wire x1="-162.56" y1="76.2" x2="-205.74" y2="76.2" width="0.1524" layer="91"/>
-<label x="-203.2" y="76.2" size="1.778" layer="95"/>
-</segment>
-</net>

Commit message: [CDH] updated trivial mismatches between connector netnames [EPS] updated trivial mismatches between connector netnames [PAYLOAD] updated trivial mismatches between connector netnames [WIRING] updated trivial mismatches between connector netnames
Connections:
- net 9V renamed POW_9V
- net BATTERY_THERMSTOR_2+ renamed BATTERY_THRMSTOR2_+V
- net BATTERY_THRMSTOR_+V renamed BATTERY_THRMSTOR1_+V
- net POW_5V renamed POW_RADIO_VBATT
- net THERMALGND renamed THERMALGND1
- removed net EXTERNAL_POWER_+V: H2.51
- removed net N$19: H2.37
- removed net N$89.: H2.21
- removed net N$90: H2.23
- removed net N$91: H2.25
- new net EXTERNAL_POWER_V+: H2.52
- new net N$1: H2.6
- new net N$6: H2.10
- new net POW_RADIO_3V3: H2.27
- new net POW_RADIO_3V3_SYS: H2.28
- net EXTERNAL_POWER_GND: now also H2.51; no longer H2.52
- net N$4: now also H2.8; no longer H2.35
- net POW_RADIO_3.3V: no longer H2.27, H2.28
- net Q6_SPI_SCLK: now also H2.21; no longer H2.6
- net Q6_SPI_SDI_MISO: now also H2.35; no longer H2.10
- net Q6_SPI_SDO_MOSI: now also H2.23; no longer H2.8
Other:
- note removed: "POW_RADIO_VBATT"

Commit message: [PAYLOAD-INT] added h2 pin 26 and pin 28 short (to match actual PCB)
Connections:
- removed net POW_RADIO_3V3_SYS: H2.28
- net POW_RADIO_3V3: now also H2.28
Changed lines of the file:
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@@
 <setting verticaltext="up"/>
 </settings>
-<grid distance="1.27" unitdist="mm" unit="mm" style="lines" multiple="1" display="no" altdistance="0.01" altunitdist="inch" altunit="mm"/>
+<grid distance="0.1" unitdist="inch" unit="inch" style="lines" multiple="1" display="no" altdistance="0.01" altunitdist="inch" altunit="inch"/>
 <layers>
 <layer number="1" name="Top" color="4" fill="1" visible="no" active="no"/>
@@
 <label x="-203.2" y="68.58" size="1.778" layer="95"/>
 </segment>
-</net>
-<net name="POW_RADIO_3V3_SYS" class="0">
 <segment>
 <pinref part="H2" gate="G$1" pin="28"/>
