File: Payload Internal - Auxiliary/Payload v2.1.sch (EAGLE design)
At the start: 11 parts

Commit message: [CDH] renamed connectors to 'J#' in sync with wiring harness [diplexer-rcl.lbr] copied rcl.lbr and created an inductor with SMD package L01005(imperial) [DIPLEXER] renamed sma connectors to 'J#' in sync with wiring harness    changed part symbols of C6 C7 C8 C9 C10 to L6 L7 L8 L9 L10 [space-concordia-power-lbr] updated 'GLENAIR-171-006-6-S-6-7-18' to have a valid prefix [Payload-Internal-Aux] renamed connectors to 'J#' in sync with wiring harness [wiring-harness] renamed all known connectors to 'J#' in sync with wiring harness
Parts:
- renumbered U$1 to J31, U$3 to J30
Changed lines of the file:
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@@
 <part name="R3" library="resistor" deviceset="R-US_" device="R2012"/>
 <part name="R4" library="resistor" deviceset="R-US_" device="R2012"/>
-<part name="U$1" library="harwin" deviceset="M80-866XXXX" device=""/>
-<part name="U$3" library="harwin" deviceset="M80-866XXXX" device=""/>
+<part name="J31" library="harwin" deviceset="M80-866XXXX" device=""/>
+<part name="J30" library="harwin" deviceset="M80-866XXXX" device=""/>
 <part name="SUPPLY1" library="supply2" deviceset="GND" device=""/>
 <part name="SUPPLY4" library="supply2" deviceset="GND" device=""/>
@@
 <instance part="R3" gate="G$1" x="-337.82" y="27.94" rot="R180"/>
 <instance part="R4" gate="G$1" x="-337.82" y="33.02" rot="R180"/>
-<instance part="U$1" gate="G$1" x="-279.4" y="55.88"/>
-<instance part="U$3" gate="G$1" x="-279.4" y="93.98"/>
+<instance part="J31" gate="G$1" x="-279.4" y="55.88"/>
+<instance part="J30" gate="G$1" x="-279.4" y="93.98"/>
 <instance part="SUPPLY1" gate="GND" x="-212.09" y="66.04" rot="R270"/>
 <instance part="SUPPLY4" gate="GND" x="-104.14" y="63.5" rot="R90"/>
@@
 </segment>
 <segment>
-<pinref part="U$3" gate="G$1" pin="14"/>
+<pinref part="J30" gate="G$1" pin="14"/>
 <wire x1="-266.7" y1="96.52" x2="-256.54" y2="96.52" width="0.1524" layer="91"/>
 <label x="-259.08" y="96.52" size="1.778" layer="95"/>
@@
 </segment>
 <segment>
-<pinref part="U$3" gate="G$1" pin="5"/>
+<pinref part="J30" gate="G$1" pin="5"/>
 <wire x1="-292.1" y1="91.44" x2="-302.26" y2="91.44" width="0.1524" layer="91"/>
 <label x="-332.74" y="91.44" size="1.778" layer="95"/>
@@
 </segment>
 <segment>
-<pinref part="U$3" gate="G$1" pin="6"/>
+<pinref part="J30" gate="G$1" pin="6"/>
 <wire x1="-292.1" y1="88.9" x2="-302.26" y2="88.9" width="0.1524" layer="91"/>
 <label x="-332.74" y="88.9" size="1.778" layer="95"/>
@@
 </segment>
 <segment>
-<pinref part="U$3" gate="G$1" pin="8"/>
+<pinref part="J30" gate="G$1" pin="8"/>
 <wire x1="-292.1" y1="83.82" x2="-302.26" y2="83.82" width="0.1524" layer="91"/>
 <label x="-332.74" y="83.82" size="1.778" layer="95"/>
@@
 </segment>
 <segment>
-<pinref part="U$3" gate="G$1" pin="2"/>
+<pinref part="J30" gate="G$1" pin="2"/>
 <wire x1="-292.1" y1="99.06" x2="-302.26" y2="99.06" width="0.1524" layer="91"/>
 <label x="-327.66" y="99.06" size="1.778" layer="95"/>
@@
 </segment>
 <segment>
-<pinref part="U$3" gate="G$1" pin="4"/>
+<pinref part="J30" gate="G$1" pin="4"/>
 <wire x1="-292.1" y1="93.98" x2="-302.26" y2="93.98" width="0.1524" layer="91"/>
 <label x="-327.66" y="93.98" size="1.778" layer="95"/>
@@
 </segment>
 <segment>
-<pinref part="U$3" gate="G$1" pin="3"/>
+<pinref part="J30" gate="G$1" pin="3"/>
 <wire x1="-292.1" y1="96.52" x2="-302.26" y2="96.52" width="0.1524" layer="91"/>
 <label x="-327.66" y="96.52" size="1.778" layer="95"/>
@@
 </segment>
 <segment>
-<pinref part="U$3" gate="G$1" pin="1"/>
+<pinref part="J30" gate="G$1" pin="1"/>
 <wire x1="-292.1" y1="101.6" x2="-302.26" y2="101.6" width="0.1524" layer="91"/>
 <label x="-327.66" y="101.6" size="1.778" layer="95"/>
@@
 </segment>
 <segment>
-<pinref part="U$3" gate="G$1" pin="7"/>
+<pinref part="J30" gate="G$1" pin="7"/>
 <wire x1="-292.1" y1="86.36" x2="-302.26" y2="86.36" width="0.1524" layer="91"/>
 <label x="-332.74" y="86.36" size="1.778" layer="95"/>
@@
 </segment>
 <segment>
-<pinref part="U$3" gate="G$1" pin="13"/>
+<pinref part="J30" gate="G$1" pin="13"/>
 <wire x1="-266.7" y1="93.98" x2="-254" y2="93.98" width="0.1524" layer="91"/>
 <label x="-259.08" y="93.98" size="1.778" layer="95"/>
@@
 </segment>
 <segment>
-<pinref part="U$3" gate="G$1" pin="12"/>
+<pinref part="J30" gate="G$1" pin="12"/>
 <wire x1="-266.7" y1="91.44" x2="-256.54" y2="91.44" width="0.1524" layer="91"/>
 <label x="-259.08" y="91.44" size="1.778" layer="95"/>
@@
 </segment>
 <segment>
-<pinref part="U$1" gate="G$1" pin="11"/>
+<pinref part="J31" gate="G$1" pin="11"/>
 <wire x1="-266.7" y1="50.8" x2="-256.54" y2="50.8" width="0.1524" layer="91"/>
 <label x="-259.08" y="50.8" size="1.778" layer="95"/>
@@
 </segment>
 <segment>
-<pinref part="U$1" gate="G$1" pin="10"/>
+<pinref part="J31" gate="G$1" pin="10"/>
 <wire x1="-266.7" y1="48.26" x2="-256.54" y2="48.26" width="0.1524" layer="91"/>
 <label x="-259.08" y="48.26" size="1.778" layer="95"/>
@@
 </segment>
 <segment>
-<pinref part="U$3" gate="G$1" pin="16"/>
+<pinref part="J30" gate="G$1" pin="16"/>
 <wire x1="-266.7" y1="101.6" x2="-256.54" y2="101.6" width="0.1524" layer="91"/>
 <label x="-259.08" y="101.6" size="1.778" layer="95"/>
@@
 </segment>
 <segment>
-<pinref part="U$3" gate="G$1" pin="15"/>
+<pinref part="J30" gate="G$1" pin="15"/>
 <wire x1="-266.7" y1="99.06" x2="-256.54" y2="99.06" width="0.1524" layer="91"/>
 <label x="-259.08" y="99.06" size="1.778" layer="95"/>
@@
 </segment>
 <segment>
-<pinref part="U$1" gate="G$1" pin="16"/>
+<pinref part="J31" gate="G$1" pin="16"/>
 <wire x1="-266.7" y1="63.5" x2="-259.08" y2="63.5" width="0.1524" layer="91"/>
 <label x="-259.08" y="63.5" size="1.778" layer="95"/>
@@
 </segment>
 <segment>
-<pinref part="U$1" gate="G$1" pin="15"/>
+<pinref part="J31" gate="G$1" pin="15"/>
 <wire x1="-266.7" y1="60.96" x2="-256.54" y2="60.96" width="0.1524" layer="91"/>
 <label x="-259.08" y="60.96" size="1.778" layer="95"/>
@@
 </segment>
 <segment>
-<pinref part="U$1" gate="G$1" pin="1"/>
+<pinref part="J31" gate="G$1" pin="1"/>
 <wire x1="-292.1" y1="63.5" x2="-299.72" y2="63.5" width="0.1524" layer="91"/>
 <label x="-327.66" y="63.5" size="1.778" layer="95"/>
@@
 </segment>
 <segment>
-<pinref part="U$1" gate="G$1" pin="3"/>
+<pinref part="J31" gate="G$1" pin="3"/>
 <wire x1="-292.1" y1="58.42" x2="-299.72" y2="58.42" width="0.1524" layer="91"/>
 <label x="-327.66" y="58.42" size="1.778" layer="95"/>
@@
 <net name="N$18" class="0">
 <segment>
-<pinref part="U$3" gate="G$1" pin="10"/>
+<pinref part="J30" gate="G$1" pin="10"/>
 <wire x1="-266.7" y1="86.36" x2="-256.54" y2="86.36" width="0.1524" layer="91"/>
 <label x="-259.08" y="86.36" size="1.778" layer="95"/>
@@
 <net name="N$20" class="0">
 <segment>
-<pinref part="U$3" gate="G$1" pin="11"/>
+<pinref part="J30" gate="G$1" pin="11"/>
 <wire x1="-266.7" y1="88.9" x2="-256.54" y2="88.9" width="0.1524" layer="91"/>
 <label x="-259.08" y="88.9" size="1.778" layer="95"/>
@@
 <net name="N$32" class="0">
 <segment>
-<pinref part="U$1" gate="G$1" pin="5"/>
+<pinref part="J31" gate="G$1" pin="5"/>
 <wire x1="-292.1" y1="53.34" x2="-299.72" y2="53.34" width="0.1524" layer="91"/>
 <label x="-299.72" y="53.34" size="1.778" layer="95"/>
@@
 <net name="N$33" class="0">
 <segment>
-<pinref part="U$1" gate="G$1" pin="6"/>
+<pinref part="J31" gate="G$1" pin="6"/>
 <wire x1="-292.1" y1="50.8" x2="-299.72" y2="50.8" width="0.1524" layer="91"/>
 <label x="-299.72" y="50.8" size="1.778" layer="95"/>
@@
 <net name="N$34" class="0">
 <segment>
-<pinref part="U$1" gate="G$1" pin="8"/>
+<pinref part="J31" gate="G$1" pin="8"/>
 <wire x1="-292.1" y1="45.72" x2="-299.72" y2="45.72" width="0.1524" layer="91"/>
 <label x="-299.72" y="45.72" size="1.778" layer="95"/>
@@
 <net name="N$35" class="0">
 <segment>
-<pinref part="U$1" gate="G$1" pin="7"/>
+<pinref part="J31" gate="G$1" pin="7"/>
 <wire x1="-292.1" y1="48.26" x2="-299.72" y2="48.26" width="0.1524" layer="91"/>
 <label x="-299.72" y="48.26" size="1.778" layer="95"/>
@@
 <net name="N$37" class="0">
 <segment>
-<pinref part="U$1" gate="G$1" pin="14"/>
+<pinref part="J31" gate="G$1" pin="14"/>
 <wire x1="-266.7" y1="58.42" x2="-259.08" y2="58.42" width="0.1524" layer="91"/>
 <label x="-259.08" y="58.42" size="1.778" layer="95"/>
@@
 <net name="N$39" class="0">
 <segment>
-<pinref part="U$1" gate="G$1" pin="13"/>
+<pinref part="J31" gate="G$1" pin="13"/>
 <wire x1="-266.7" y1="55.88" x2="-256.54" y2="55.88" width="0.1524" layer="91"/>
 <label x="-259.08" y="55.88" size="1.778" layer="95"/>
@@
 </segment>
 <segment>
-<pinref part="U$3" gate="G$1" pin="9"/>
+<pinref part="J30" gate="G$1" pin="9"/>
 <wire x1="-266.7" y1="83.82" x2="-256.54" y2="83.82" width="0.1524" layer="91"/>
 <label x="-259.08" y="83.82" size="1.778" layer="95"/>
@@
 <net name="PAYGND" class="0">
 <segment>
-<pinref part="U$1" gate="G$1" pin="9"/>
+<pinref part="J31" gate="G$1" pin="9"/>
 <wire x1="-266.7" y1="45.72" x2="-256.54" y2="45.72" width="0.1524" layer="91"/>
 <label x="-259.08" y="45.72" size="1.778" layer="95"/>
@@
 </segment>
 <segment>
-<pinref part="U$1" gate="G$1" pin="12"/>
+<pinref part="J31" gate="G$1" pin="12"/>
 <wire x1="-266.7" y1="53.34" x2="-256.54" y2="53.34" width="0.1524" layer="91"/>
 <label x="-259.08" y="53.34" size="1.778" layer="95"/>
@@
 </segment>
 <segment>
-<pinref part="U$1" gate="G$1" pin="2"/>
+<pinref part="J31" gate="G$1" pin="2"/>
 <wire x1="-292.1" y1="60.96" x2="-299.72" y2="60.96" width="0.1524" layer="91"/>
 <label x="-327.66" y="60.96" size="1.778" layer="95"/>
@@
 </segment>
 <segment>
-<pinref part="U$1" gate="G$1" pin="4"/>
+<pinref part="J31" gate="G$1" pin="4"/>
 <wire x1="-292.1" y1="55.88" x2="-299.72" y2="55.88" width="0.1524" layer="91"/>
 <label x="-327.66" y="55.88" size="1.778" layer="95"/>

Commit message: [CDH] [Wiring Harness] [Payload-Internal-Aux] renamed nets 'Q6_PC_RS232' and 'PC_Q6_RS232' to 'Q6_MAX_RS232' and 'MAX_Q6_RS232' for clarity
Connections:
- net PC_Q6_RS232 renamed MAX_Q6_RS232
- net Q6_PC_RS232 renamed Q6_MAX_RS232
Changed lines of the file:
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@@
 <?xml version="1.0" encoding="utf-8"?>
 <!DOCTYPE eagle SYSTEM "eagle.dtd">
-<eagle version="7.2.0">
+<eagle version="7.3.0">
 <drawing>
 <settings>
@@
 </segment>
 </net>
-<net name="PC_Q6_RS232" class="0">
+<net name="MAX_Q6_RS232" class="0">
 <segment>
 <pinref part="H1" gate="G$1" pin="21"/>
@@
 </segment>
 </net>
-<net name="Q6_PC_RS232" class="0">
+<net name="Q6_MAX_RS232" class="0">
 <segment>
 <pinref part="H1" gate="G$1" pin="25"/>

Commit message: [Wiring Harness] [Payload-Internal-Aux] Renamed unconnected header pins to match wiring harness. The remaining conflicts are legitimate wired net conflicts and can only be resolved with redesign.
Connections:
- net 9V renamed POW_9V
- net BATTERY_THERMSTOR_2+ renamed BATTERY_THRMSTOR2_+V
- net POW_RADIO_3.3V renamed POW_RADIO_3V3SYS
- net THERMALGND renamed THERMALGND1
- removed net N$89.: H2.21
- removed net N$90: H2.23
- new net N$1: H2.6
- new net N$6: H2.10
- net EXTERNAL_POWER_+V: now also H2.52; no longer H2.51
- net EXTERNAL_POWER_GND: now also H2.51; no longer H2.52
- net N$4: now also H2.8; no longer H2.35
- net Q6_SPI_SCLK: now also H2.21; no longer H2.6
- net Q6_SPI_SDI_MISO: now also H2.35; no longer H2.10
- net Q6_SPI_SDO_MOSI: now also H2.23; no longer H2.8
Changed lines of the file:
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@@
 </segment>
 </net>
-<net name="N$90" class="0">
+<net name="Q6_SPI_SDO_MOSI" class="0">
 <segment>
 <pinref part="H2" gate="G$1" pin="23"/>
@@
 </segment>
 </net>
-<net name="Q6_SPI_SDO_MOSI" class="0">
+<net name="N$4" class="0">
 <segment>
 <wire x1="-139.7" y1="93.98" x2="-106.68" y2="93.98" width="0.1524" layer="91"/>
@@
 <net name="Q6_SPI_CS1" class="0">
 <segment>
+<pinref part="R8" gate="G$1" pin="1"/>
+<wire x1="-332.74" y1="7.62" x2="-327.66" y2="7.62" width="0.1524" layer="91"/>
+<label x="-325.12" y="7.62" size="1.778" layer="95"/>
+</segment>
+<segment>
 <wire x1="-139.7" y1="88.9" x2="-107.95" y2="88.9" width="0.1524" layer="91"/>
 <pinref part="H2" gate="G$1" pin="12"/>
 <label x="-137.16" y="88.9" size="1.778" layer="95"/>
-</segment>
-<segment>
-<pinref part="R8" gate="G$1" pin="1"/>
-<wire x1="-332.74" y1="7.62" x2="-327.66" y2="7.62" width="0.1524" layer="91"/>
-<label x="-325.12" y="7.62" size="1.778" layer="95"/>
 </segment>
 </net>
@@
 </segment>
 </net>
-<net name="N$89." class="0">
+<net name="Q6_SPI_SCLK" class="0">
 <segment>
 <pinref part="H2" gate="G$1" pin="21"/>
@@
 </segment>
 </net>
-<net name="Q6_SPI_SCLK" class="0">
+<net name="N$1" class="0">
 <segment>
 <pinref part="H2" gate="G$1" pin="6"/>
@@
 </segment>
 </net>
-<net name="Q6_SPI_SDI_MISO" class="0">
+<net name="N$6" class="0">
 <segment>
 <pinref part="H2" gate="G$1" pin="10"/>
@@
 </segment>
 </net>
-<net name="POW_RADIO_3.3V" class="0">
+<net name="POW_RADIO_3V3SYS" class="0">
 <segment>
 <pinref part="H2" gate="G$1" pin="27"/>
@@
 </segment>
 </net>
-<net name="N$4" class="0">
+<net name="Q6_SPI_SDI_MISO" class="0">
 <segment>
 <pinref part="H2" gate="G$1" pin="35"/>
@@
 </segment>
 </net>
-<net name="EXTERNAL_POWER_GND" class="0">
+<net name="EXTERNAL_POWER_+V" class="0">
 <segment>
 <pinref part="H2" gate="G$1" pin="52"/>
@@
 </segment>
 </net>
-<net name="EXTERNAL_POWER_+V" class="0">
+<net name="EXTERNAL_POWER_GND" class="0">
 <segment>
 <pinref part="H2" gate="G$1" pin="51"/>
@@
 </segment>
 </net>
-<net name="THERMALGND" class="0">
+<net name="THERMALGND1" class="0">
 <segment>
 <pinref part="H1" gate="G$1" pin="5"/>
@@
 </segment>
 </net>
-<net name="9V" class="0">
+<net name="POW_9V" class="0">
 <segment>
 <pinref part="H1" gate="G$1" pin="22"/>
@@
 </segment>
 </net>
-<net name="N$6546" class="0">
+<net name="N$654643543" class="0">
 <segment>
 <pinref part="H1" gate="G$1" pin="14"/>
@@
 </segment>
 </net>
-<net name="BATTERY_THERMSTOR_2+" class="0">
+<net name="BATTERY_THRMSTOR2_+V" class="0">
 <segment>
 <pinref part="H1" gate="G$1" pin="12"/>

Commit message: [Payload-Internal-Aux] During 20160705 unit testing it was noticed that pin9(vcc) and pin10(!forceoff) were shorted. Updated schematic to match.
Connections:
- net +3V3: now also U$8.~FORCEOFF
Changed lines of the file:
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@@
 <pinref part="U$8" gate="G$1" pin="VCC"/>
 <junction x="-236.22" y="-20.32"/>
+<pinref part="U$8" gate="G$1" pin="~FORCEOFF"/>
+<wire x1="-302.26" y1="-45.72" x2="-302.26" y2="-53.34" width="0.1524" layer="91"/>
+<wire x1="-302.26" y1="-53.34" x2="-236.22" y2="-53.34" width="0.1524" layer="91"/>
+<wire x1="-236.22" y1="-53.34" x2="-236.22" y2="-20.32" width="0.1524" layer="91"/>
 </segment>
 <segment>
