File: Payload Internal - Auxiliary/Auxiliary-Payload v4.2.brd (EAGLE design)
At the start: 90.5 x 91.8 mm, 101 parts, among them IC2 ATMEGA328P-AU, U1 AD7294BSUZ

Commit message: Update payload internal to version 4.2
Parts:
- removed U$10, U$11, U$12, U$13, U$14, U$15, U$16, U$17, U$18, U$19, U$27, U$28, U$32, U$35, U$37, U$7, U$9: CONNECTOR-SHORT, Payload-board:CONNECTOR-T
- removed U$20, U$22, U$23, U$24: CONNECTOR-3, Payload-board:CONNECTOR-3T
- removed U$21, U$25: CONNECTOR-4, Payload-board:CONNECTOR-4T
- added C27, C32, C34: 51 pF, rcl:C0603
- added C28, C31, C35: 0.1 uF, rcl:C0603
- added C29, C33, C36: 10 uF, rcl:C1210
- added C30: 15 pF, rcl:C0603
- added R32, R33: 500 Ohm, rcl:R0805
- added R34: 3.5 MOhm, rcl:R1206
- added R35: 178 Ohm, rcl:R1210
- C1: value (none) -> 100 nF
- C10, C11, C20, C22, C23, C24, C25, C7: value (none) -> 10 uF
- C12, C13, C14, C15, C16, C17, C18, C2, C21, C8, C9: value (none) -> 0.1 uF
- C19, C26: value (none) -> 51 pF
- C3, C6: value (none) -> 10 uF; device rcl:C1206 -> rcl:C1210
- C4, C5: value (none) -> 22 pF
- R11, R5: value (none) -> 1 MOhm
- R12, R6: value (none) -> 36 Ohm
- R13, R14: value (none) -> 100 kOhm
- R15: value (none) -> 178 Ohm
- R16: value (none) -> 1.4 MOhm
- R17, R19, R2, R22, R7: value (none) -> 1 kOhm
- R18, R20: value (none) -> 1.5 MOhm
- R21, R23, R24, R25, R26, R27, R28, R29, R30: value (none) -> 100 Ohm
- R3, R4, R8, R9: value (none) -> 4.7 kOhm
- R31: value (none) -> 10 kOhm
- U$6: value CONNECTOR-SHORT -> 74LVC1G18-SOT363; device Payload-board:CONNECTOR-T -> Payload-board:SOT-363
- moved U$6 57.2 mm to (81.0, 29.2), turned to 90 degrees
- moved U$36 47.4 mm to (37.6, 69.4), turned to 0 degrees
- moved C19 27.9 mm to (56.9, 43.5)
- moved U$38 18.7 mm to (63.7, 37.6), turned to 180 degrees
- moved C26 14.8 mm to (65.1, 42.7)
- moved U$34 5.95 mm to (35.1, 69.6), turned to 90 degrees
- moved C25 5.92 mm to (46.6, 26.4), turned to 270 degrees
- moved R19 2.06 mm to (77.3, 26.2)
- moved U$33 1.16 mm to (83.0, 81.8)
- moved R18 0.32 mm to (88.0, 23.9)
- moved C18 0.21 mm to (43.1, 28.2), turned to 90 degrees
Connections:
- removed net N$12: R28.1, U$24.P$3
- removed net N$14: C22.+, U$21.P$4
- removed net N$16: R27.2, U$23.P$3
- removed net N$17: C25.+, U$25.P$4
- removed net N$24: R26.1, U$22.P$3
- removed net N$25: R25.2, U$20.P$3
- removed net PS1+: U$37.P$1, U1.62
- removed net PS2+: U$35.P$1, U1.63
- removed net REFINADC: U$25.P$3
- removed net REFINDAC: U$21.P$3
- removed net VCCA: C26.1, U$38.1
- removed net VCCY: C19.1, U$38.14
- new net A: R34.2, R35.2, U$6.P$3
- new net DEMUX_VCC: C35.2, C36.2, U$6.P$5
- net +3V3: now also C31.1, C33.1, U$38.1, U$38.8
- net AGND_ADC: no longer U$10.P$2, U$11.P$2, U$12.P$2, U$13.P$1, U$14.P$1, U$15.P$1, U$16.P$1, U$17.P$2, U$18.P$2, U$19.P$2, U$20.P$2, U$21.P$2, U$22.P$2, U$23.P$2, U$24.P$2, U$25.P$2, U$27.P$2, U$35.P$2, U$37.P$2, U$6.P$2, U$7.P$2, U$9.P$2
- net D1(+): now also R25.2; no longer U$20.P$1
- net D1(-): now also R26.1; no longer U$22.P$1
- net D2(+): now also R27.2; no longer U$23.P$1
- net D2(-): now also R28.1; no longer U$24.P$1
- net DGND_ADC: no longer U$28.P$2
- net GND: now also U$34.P$1, U$36.P$1; no longer U$32.P$1
- net GND1: now also C27.2, C28.2, C29.2, C30.2, C31.2, C32.1, C33.2, C34.2, R32.2, R33.1, R34.1, U$38.7, U$6.P$2; no longer U$32.P$2, U$34.P$1, U$36.P$1
- net IO3: now also R35.1
- net IO9: now also U$6.P$1
- net ISENSE1OVERRANGE: no longer U$12.P$1
- net ISENSE2OVERRANGE: no longer U$27.P$1
- net N$19: now also U$38.5
- net N$3: now also U$38.13
- net N$4: now also C30.1, U$38.2
- net N$51: now also C27.1, U$38.12
- net N$89.: now also U$38.4
- net N$90: now also U$38.3
- net OFFSETINA: no longer U$6.P$1
- net OFFSETINB: no longer U$9.P$1
- net OFFSETINC: no longer U$10.P$1
- net OFFSETIND: no longer U$11.P$1
- net POW_5V: now also C28.1, C29.1, C35.1, C36.1, U$38.14; no longer U$28.P$1
- net PULSE1: now also C32.2, R32.1, U$6.P$6
- net PULSE2: now also C34.1, R33.2, U$6.P$4
- net REFOUT/REFINADC: now also C25.+; no longer U$25.P$1
- net REFOUT/REFINDAC: now also C22.+; no longer U$21.P$1
- net RS1+: now also U1.62; no longer U$15.P$2
- net RS1-: no longer U$16.P$2
- net RS2+: now also U1.63; no longer U$13.P$2
- net RS2-: no longer U$14.P$2
- net SCK: now also C19.1, U$38.11
- net SS: now also C26.1, U$38.10
- net VOUTA: no longer U$17.P$1
- net VOUTB: no longer U$7.P$1
- net VOUTC: no longer U$18.P$1
- net VOUTD: no longer U$19.P$1
Routing:
- net +3V3: track 80.8 -> 208.1 mm, vias 0 -> 6
- net SOLAR_PANEL_2_4: track 0.00 -> 125.7 mm, vias 0 -> 3
- net ANTENNA_DEPLOYMENT_+V: track 3.32 -> 105.3 mm, vias 0 -> 2
- net AGND_ADC: track 276.8 -> 181.3 mm, vias 11 -> 9
- net ANTENNA_DEPLOYMENT_GND: track 0.00 -> 94.8 mm, vias 0 -> 6
- net GND1: track 88.7 -> 175.7 mm, vias 16 -> 17
- net G-M-OUTPUT-AMPLITUDE: track 6.83 -> 90.5 mm
- net GND3: track 0.00 -> 82.5 mm, vias 0 -> 6
- net PULSE2: track 0.00 -> 78.9 mm, vias 0 -> 2
- net N$19: track 0.00 -> 77.8 mm, vias 0 -> 3
- net SCK: track 20.2 -> 95.9 mm, vias 0 -> 2
- net HV_OUTPUT2: track 3.69 -> 78.0 mm, vias 1 -> 3
- net N$4: track 0.00 -> 73.7 mm, vias 0 -> 3
- net HV_OUTPUT1: track 12.7 -> 84.7 mm, vias 0 -> 3
- net N$89.: track 0.00 -> 69.9 mm, vias 0 -> 1
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