File: Payload Internal - Auxiliary/Auxiliary-Payload v4.2.sch (EAGLE design)
At the start: 101 parts, among them IC2 ATMEGA328P-AU, U1 AD7294BSUZ

Commit message: Update payload internal to version 4.2
Parts:
- removed U$10, U$11, U$12, U$13, U$14, U$15, U$16, U$17, U$18, U$19, U$27, U$28, U$32, U$35, U$37, U$7, U$9: CONNECTOR-SHORT, Payload-board:CONNECTOR-SHORT
- removed U$20, U$22, U$23, U$24: CONNECTOR-3, Payload-board:CONNECTOR-3
- removed U$21, U$25: CONNECTOR-4, Payload-board:CONNECTOR-4
- added C27: 51 pF, rcl:C-USC0603
- added C28, C31, C35: 0.1 uF, rcl:C-USC0603
- added C29, C33, C36: 10 uF, rcl:C-USC1210
- added C30: 15 pF, rcl:C-USC0603
- added C32, C34: 51 pF, rcl:C-EUC0603
- added R32, R33: 500 Ohm, rcl:R-US_R0805
- added R34: 3.5 MOhm, rcl:R-US_R1206
- added R35: 178 Ohm, rcl:R-US_R1210
- C1: value (none) -> 100 nF
- C10, C11, C20, C22, C23, C24, C25, C7: value (none) -> 10 uF
- C12, C13, C14, C15, C16, C17, C18, C2, C21, C8, C9: value (none) -> 0.1 uF
- C19, C26: value (none) -> 51 pF; device rcl:C-EUC0603 -> rcl:C-USC0603
- C3, C6: value (none) -> 10 uF; device rcl:C-EUC1206 -> rcl:C-USC1210
- C4, C5: value (none) -> 22 pF
- R11, R5: value (none) -> 1 MOhm
- R12, R6: value (none) -> 36 Ohm
- R13, R14: value (none) -> 100 kOhm
- R15: value (none) -> 178 Ohm
- R16: value (none) -> 1.4 MOhm
- R17, R19, R2, R22, R7: value (none) -> 1 kOhm
- R18, R20: value (none) -> 1.5 MOhm
- R21, R23, R24, R25, R26, R27, R28, R29, R30: value (none) -> 100 Ohm
- R3, R4, R8, R9: value (none) -> 4.7 kOhm
- R31: value (none) -> 10 kOhm
- U$6: value CONNECTOR-SHORT -> 74LVC1G18-SOT363; device Payload-board:CONNECTOR-SHORT -> Payload-board:74LVC1G18-SOT363
Connections:
- removed net N$12: R28.1, U$24.3
- removed net N$14: C22.+, U$21.4
- removed net N$16: R27.2, U$23.3
- removed net N$17: C25.+, U$25.4
- removed net N$24: R26.1, U$22.3
- removed net N$25: R25.2, U$20.3
- removed net PS1+: U$37.IN, U1.VPP1
- removed net PS2+: U$35.IN, U1.VPP2
- removed net REFINADC: U$25.3
- removed net REFINDAC: U$21.3
- removed net VCCA: C26.1, U$38.VCCA
- removed net VCCY: C19.1, U$38.VCCY
- new net A: R34.2, R35.2, U$6.A
- new net DEMUX_VCC: C35.2, C36.2, U$6.VCC
- net +3V3: now also C31.1, C33.1, U$38.EN, U$38.VCCA
- net AGND_ADC: no longer U$10.OUT, U$11.OUT, U$12.OUT, U$13.IN, U$14.IN, U$15.IN, U$16.IN, U$17.OUT, U$18.OUT, U$19.OUT, U$20.2, U$21.2, U$22.2, U$23.2, U$24.2, U$25.2, U$27.OUT, U$35.OUT, U$37.OUT, U$6.OUT, U$7.OUT, U$9.OUT
- net D1(+): now also R25.2; no longer U$20.1
- net D1(-): now also R26.1; no longer U$22.1
- net D2(+): now also R27.2; no longer U$23.1
- net D2(-): now also R28.1; no longer U$24.1
- net DGND_ADC: no longer U$28.OUT
- net GND: now also U$34.IN, U$36.IN; no longer U$32.IN
- net GND1: now also C27.2, C28.2, C29.2, C30.2, C31.2, C32.1, C33.2, C34.2, R32.2, R33.1, R34.1, U$38.GND, U$6.GND; no longer U$32.OUT, U$34.IN, U$36.IN
- net IO3: now also R35.1
- net IO9: now also U$6.S
- net ISENSE1OVERRANGE: no longer U$12.IN
- net ISENSE2OVERRANGE: no longer U$27.IN
- net N$19: now also U$38.A4
- net N$3: now also U$38.Y1
- net N$4: now also C30.1, U$38.A1
- net N$51: now also C27.1, U$38.Y2
- net N$89.: now also U$38.A3
- net N$90: now also U$38.A2
- net OFFSETINA: no longer U$6.IN
- net OFFSETINB: no longer U$9.IN
- net OFFSETINC: no longer U$10.IN
- net OFFSETIND: no longer U$11.IN
- net POW_5V: now also C28.1, C29.1, C35.1, C36.1, U$38.VCCY; no longer U$28.IN
- net PULSE1: now also C32.2, R32.1, U$6.1Y
- net PULSE2: now also C34.1, R33.2, U$6.2Y
- net REFOUT/REFINADC: now also C25.+; no longer U$25.1
- net REFOUT/REFINDAC: now also C22.+; no longer U$21.1
- net RS1+: now also U1.VPP1; no longer U$15.OUT
- net RS1-: no longer U$16.OUT
- net RS2+: now also U1.VPP2; no longer U$13.OUT
- net RS2-: no longer U$14.OUT
- net SCK: now also C19.1, U$38.Y3
- net SS: now also C26.1, U$38.Y4
- net VOUTA: no longer U$17.IN
- net VOUTB: no longer U$7.IN
- net VOUTC: no longer U$18.IN
- net VOUTD: no longer U$19.IN
Other:
- note removed: "DAC voltage connected to ground"
- moved on the sheet: C19, C22, C25, C26, C7, C8, U$38

Commit message: worked on the wiring harness:   - fixed some signals between ext payload and int payload   - added wire data.ods sheet
ran 'snap to grid' on internal payload schematic
Other:
- moved on the sheet: C1, C11, C15, C16, C17, C18, C21, C26, C28, C29, C32, C34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
