File: Payload Internal - Auxiliary/Payload v2.1.brd (EAGLE design)
At the start: 90.5 x 91.8 mm, 11 parts

Commit message: [CDH] renamed connectors to 'J#' in sync with wiring harness [diplexer-rcl.lbr] copied rcl.lbr and created an inductor with SMD package L01005(imperial) [DIPLEXER] renamed sma connectors to 'J#' in sync with wiring harness    changed part symbols of C6 C7 C8 C9 C10 to L6 L7 L8 L9 L10 [space-concordia-power-lbr] updated 'GLENAIR-171-006-6-S-6-7-18' to have a valid prefix [Payload-Internal-Aux] renamed connectors to 'J#' in sync with wiring harness [wiring-harness] renamed all known connectors to 'J#' in sync with wiring harness
Parts:
- renumbered U$1 to J31, U$3 to J30

Commit message: [CDH] [Wiring Harness] [Payload-Internal-Aux] renamed nets 'Q6_PC_RS232' and 'PC_Q6_RS232' to 'Q6_MAX_RS232' and 'MAX_Q6_RS232' for clarity
Connections:
- net PC_Q6_RS232 renamed MAX_Q6_RS232
- net Q6_PC_RS232 renamed Q6_MAX_RS232
Changed lines of the file:
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@@
 <?xml version="1.0" encoding="utf-8"?>
 <!DOCTYPE eagle SYSTEM "eagle.dtd">
-<eagle version="7.2.0">
+<eagle version="7.3.0">
 <drawing>
 <settings>
@@
 <contactref element="H1" pad="7"/>
 </signal>
-<signal name="PC_Q6_RS232">
+<signal name="MAX_Q6_RS232">
 <contactref element="H1" pad="21"/>
 <contactref element="U$8" pad="7"/>
@@
 <wire x1="39.72488125" y1="76.414978125" x2="39.6954" y2="76.444459375" width="0.4064" layer="16"/>
 </signal>
-<signal name="Q6_PC_RS232">
+<signal name="Q6_MAX_RS232">
 <contactref element="H1" pad="25"/>
 <contactref element="U$8" pad="8"/>

Commit message: [Wiring Harness] [Payload-Internal-Aux] Renamed unconnected header pins to match wiring harness. The remaining conflicts are legitimate wired net conflicts and can only be resolved with redesign.
Connections:
- net 9V renamed POW_9V
- net BATTERY_THERMSTOR_2+ renamed BATTERY_THRMSTOR2_+V
- net POW_RADIO_3.3V renamed POW_RADIO_3V3SYS
- net THERMALGND renamed THERMALGND1
- removed net N$89.: H2.21
- removed net N$90: H2.23
- new net N$1: H2.6
- new net N$6: H2.10
- net EXTERNAL_POWER_+V: now also H2.52; no longer H2.51
- net EXTERNAL_POWER_GND: now also H2.51; no longer H2.52
- net N$4: now also H2.8; no longer H2.35
- net Q6_SPI_SCLK: now also H2.21; no longer H2.6
- net Q6_SPI_SDI_MISO: now also H2.35; no longer H2.10
- net Q6_SPI_SDO_MOSI: now also H2.23; no longer H2.8
Changed lines of the file:
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@@
 <contactref element="H2" pad="34"/>
 </signal>
-<signal name="N$90">
+<signal name="Q6_SPI_SDO_MOSI">
 <contactref element="H2" pad="23"/>
 </signal>
@@
 <contactref element="H1" pad="33"/>
 </signal>
-<signal name="Q6_SPI_SDO_MOSI">
+<signal name="N$4">
 <contactref element="H2" pad="8"/>
 </signal>
 <signal name="Q6_SPI_CS1">
-<contactref element="H2" pad="12"/>
 <contactref element="R8" pad="1"/>
-<wire x1="27.116940625" y1="89.05731875" x2="27.116940625" y2="88.762053125" width="0.4064" layer="16"/>
 <wire x1="27.116940625" y1="88.762053125" x2="26.092159375" y2="87.737271875" width="0.4064" layer="16"/>
 <wire x1="26.092159375" y1="87.737271875" x2="13.38401875" y2="87.737271875" width="0.4064" layer="16"/>
@@
 <wire x1="20.735734375" y1="34.61491875" x2="20.735734375" y2="38.376096875" width="0.4064" layer="1"/>
 <wire x1="20.735734375" y1="38.376096875" x2="20.639834375" y2="38.471996875" width="0.4064" layer="1"/>
+<contactref element="H2" pad="12"/>
+<wire x1="27.116940625" y1="88.762053125" x2="27.116940625" y2="89.05731875" width="0.4064" layer="16"/>
 </signal>
 <signal name="Q6_GPIO_7">
@@
 <wire x1="81.331828125" y1="77.2444875" x2="82.066653125" y2="76.5096625" width="0.4064" layer="1"/>
 </signal>
-<signal name="N$89.">
+<signal name="Q6_SPI_SCLK">
 <contactref element="H2" pad="21"/>
 </signal>
-<signal name="Q6_SPI_SCLK">
+<signal name="N$1">
 <contactref element="H2" pad="6"/>
 </signal>
-<signal name="Q6_SPI_SDI_MISO">
+<signal name="N$6">
 <contactref element="H2" pad="10"/>
 </signal>
@@
 <contactref element="H2" pad="25"/>
 </signal>
-<signal name="POW_RADIO_3.3V">
+<signal name="POW_RADIO_3V3SYS">
 <contactref element="H2" pad="27"/>
 <contactref element="H1" pad="16"/>
@@
 <contactref element="H2" pad="49"/>
 </signal>
-<signal name="N$4">
+<signal name="Q6_SPI_SDI_MISO">
 <contactref element="H2" pad="35"/>
 </signal>
-<signal name="EXTERNAL_POWER_GND">
+<signal name="EXTERNAL_POWER_+V">
 <contactref element="H2" pad="52"/>
 </signal>
@@
 <contactref element="H1" pad="13"/>
 </signal>
-<signal name="EXTERNAL_POWER_+V">
+<signal name="EXTERNAL_POWER_GND">
 <contactref element="H2" pad="51"/>
 </signal>
@@
 <contactref element="J31" pad="13"/>
 </signal>
-<signal name="THERMALGND">
+<signal name="THERMALGND1">
 <contactref element="H1" pad="5"/>
 <contactref element="J30" pad="9"/>
@@
 <contactref element="J31" pad="9"/>
 </signal>
-<signal name="N$6">
+<signal name="N$60">
 <via x="9.062225" y="88.85175625" extent="1-16" drill="3.3"/>
 </signal>
@@
 <via x="85.261796875" y="3.130459375" extent="1-16" drill="3.3"/>
 </signal>
-<signal name="N$9">
+<signal name="N$61">
 <via x="5.259753125" y="3.12559375" extent="1-16" drill="3.3"/>
 </signal>
-<signal name="9V">
+<signal name="POW_9V">
 <contactref element="H1" pad="22"/>
 <contactref element="H1" pad="24"/>
@@
 <wire x1="45.01678125" y1="51.72485625" x2="45.1386375" y2="51.8467125" width="0.4064" layer="1"/>
 </signal>
-<signal name="N$6546">
+<signal name="N$654643543">
 <contactref element="H1" pad="14"/>
 </signal>
@@
 <wire x1="85.8217125" y1="50.10553125" x2="85.057015625" y2="50.10553125" width="0.4064" layer="1"/>
 </signal>
-<signal name="BATTERY_THERMSTOR_2+">
+<signal name="BATTERY_THRMSTOR2_+V">
 <contactref element="H1" pad="12"/>
 </signal>

Commit message: [Payload-Internal-Aux] During 20160705 unit testing it was noticed that pin9(vcc) and pin10(!forceoff) were shorted. Updated schematic to match.
Connections:
- net +3V3: now also U$8.10
Routing:
- net +3V3: track 171.7 -> 173.0 mm
Changed lines of the file:
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@@
 <vertex x="0.32268125" y="91.711446875"/>
 </polygon>
+<contactref element="U$8" pad="10"/>
+<wire x1="18.91221875" y1="48.56219375" x2="20.18221875" y2="48.56219375" width="0.4064" layer="1"/>
 </signal>
 <signal name="POW_5V">
