File: EPS/eps-v1-1.brd (EAGLE design)
At the start: 90.5 x 91.8 mm, 84 parts, among them IC1 MIC79110, IC10 MAX4374-10UMAX, IC11 TLV70228DBV, IC2 MIC79110, IC3 LT3872, IC4 LT3872, IC5 INA291-D, IC6 NCS2202, IC7 NCS2202, IC8 TLV70233DBVR, IC9 AD7998, Q1 SI7448DP, Q2 SI7448DP, Q3 SI7448DP, Q4 SI7485DP, Q6 SI7485DP, Q8 SI7485DP, Q9 SI7448DP

Commit message: brought in version 1.1 of the EPS
Parts:
- removed R11, R28: 20k, resistor:M1206
- added C17, C18, C22, C24, C25: 1uF, rcl:C0805
- added C23, C26: 0.1uF, rcl:C0805
- added IC12: TLV70233DBVR, space-concordia-power:SOT23-5
- IC6, IC7: value NCS2202 -> LT1716
- moved C19 4.40 mm to (53.0, 51.9)
- moved C20 4.37 mm to (51.1, 51.9)
- moved IC9 4.37 mm to (46.4, 50.4)
- moved R12 4.37 mm to (38.9, 47.9)
- moved R33 4.37 mm to (44.5, 44.0)
- moved R34 4.37 mm to (51.0, 43.9)
- moved R35 4.37 mm to (34.8, 52.1)
- moved R36 4.37 mm to (31.5, 53.9)
- moved IC11 1.87 mm to (71.4, 74.7)
- moved IC7 1.64 mm to (44.5, 31.0)
- moved IC8 1.43 mm to (40.2, 74.5)
- moved IC6 1.15 mm to (30.0, 30.4)
Connections:
- net N$11 renamed 9V_REG_OP_H1-22
- net N$13 renamed 3V3_CTL_H1-40
- net N$15 renamed SOLAR_PANEL_2_4_H1-2
- net N$2 renamed BATTERY_THRMSTOR2_+V_H1-12
- net N$34 renamed SOLAR_PANEL_1_3_H1-29
- net N$36 renamed ANT_CTL_H1-38
- net N$4 renamed BATTERY_HEATER_-V_H1-6
- net N$41 renamed Q6_I2C_SDA_1_H2-18
- net N$42 renamed Q6_I2C_SCL_1_H2-20
- net N$49 renamed Q6_GPIO_10_H1-50
- net N$5 renamed 9V_CTL_H1-36
- net N$50 renamed BATTERY_THRMSTOR1_+V_H1-8
- removed net N$44: H1.16, H1.20, IC8.5
- removed net N$52: IC6.1, Q9.P$4-G, R28.1
- removed net N$58: C14.1, C19.1, C20.1, H2.36, IC5.5, IC9.P$2, IC9.P$5, IC9.P$6, R38.2
- new net 3V3_REG_OP_H1-16: C24.1, H1.16, H1.20, IC8.5
- new net 5V_REG_OP_H1-26: C15.1, C16.1, C22.1, C23.1, C25.1, C26.1, H1.26, H1.28, IC10.P$9, IC12.1, IC12.3, IC6.5, IC7.5, IC8.1, R2.2, R25.2, R26.2, R3.2, R37.1
- new net N$2: H2.2, IC1.P$3, IC1.P$4, IC2.P$3, IC2.P$4, R18.2, R22.2
- new net N$45: IC6.1, Q9.P$4-G
- new net Q6_3V3_H2-36: C14.1, H2.36, IC5.5, R38.2
- net GNDA: now also C17.2, C18.2, C22.2, C23.2, C24.2, C25.2, C26.2, IC12.2, IC6.2, IC7.2; no longer IC6.5, IC7.5
- net N$18: now also C19.1, C20.1, IC12.5, IC9.P$2, IC9.P$5, IC9.P$6; no longer C15.1, C16.1, H1.26, H1.28, IC10.P$9, IC6.2, IC7.2, IC8.1, R11.2, R2.2, R25.2, R26.2, R28.2, R3.2, R37.1
- net N$33: no longer R11.1
- net N$43: now also C18.1; no longer IC1.P$3, IC1.P$4, IC2.P$3, IC2.P$4, R18.2, R22.2
- net N$47: now also C17.1
Routing:
- net 5V_REG_OP_H1-26: track 0.00 -> 197.4 mm, vias 0 -> 12
- net N$18: track 165.0 -> 19.8 mm, vias 10 -> 0
- net N$2: track 0.00 -> 131.6 mm, vias 0 -> 1
- net N$58: track 112.7 -> 0.00 mm, vias 4 -> 0
- net Q6_3V3_H2-36: track 0.00 -> 88.8 mm, vias 0 -> 3
- net N$43: track 275.5 -> 219.2 mm
- net N$52: track 46.6 -> 0.00 mm, vias 2 -> 0
- net N$45: track 0.47 -> 43.1 mm, vias 0 -> 2
- net GNDA: track 943.8 -> 982.1 mm, vias 25 -> 26
- net N$44: track 17.8 -> 0.00 mm
- net 3V3_REG_OP_H1-16: track 0.00 -> 17.4 mm
- net N$47: track 10.7 -> 17.3 mm
- net Q6_I2C_SDA_1_H2-18: track 49.6 -> 54.5 mm
- net Q6_I2C_SCL_1_H2-20: track 53.4 -> 58.0 mm
- net SOLAR_PANEL_2_4_H1-2: track 120.3 -> 115.6 mm
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