File: EPS/eps-v1-1.sch (EAGLE design)
At the start: 84 parts, among them IC1 MIC79110, IC10 MAX4374-10UMAX, IC11 TLV70228DBV, IC2 MIC79110, IC3 LT3872, IC4 LT3872, IC5 INA291-D, IC6 NCS2202, IC7 NCS2202, IC8 TLV70233DBVR, IC9 AD7998, Q1 SI7448DP, Q2 SI7448DP, Q3 SI7448DP, Q4 SI7485DP, Q6 SI7485DP, Q8 SI7485DP, Q9 SI7448DP

Commit message: brought in version 1.1 of the EPS
Parts:
- removed R11, R28: 20k, resistor:R-US_M1206
- added C17, C18, C22, C24, C25: 1uF, rcl:C-USC0805
- added C23, C26: 0.1uF, rcl:C-USC0805
- added IC12: TLV70233DBVR, space-concordia-power:TLV70233DBVR
- IC6, IC7: value NCS2202 -> LT1716; device space-concordia-power:NCS2202 -> space-concordia-power:LT1716
Connections:
- net N$11 renamed 9V_REG_OP_H1-22
- net N$13 renamed 3V3_CTL_H1-40
- net N$15 renamed SOLAR_PANEL_2_4_H1-2
- net N$2 renamed BATTERY_THRMSTOR2_+V_H1-12
- net N$34 renamed SOLAR_PANEL_1_3_H1-29
- net N$36 renamed ANT_CTL_H1-38
- net N$4 renamed BATTERY_HEATER_-V_H1-6
- net N$41 renamed Q6_I2C_SDA_1_H2-18
- net N$42 renamed Q6_I2C_SCL_1_H2-20
- net N$49 renamed Q6_GPIO_10_H1-50
- net N$5 renamed 9V_CTL_H1-36
- net N$50 renamed BATTERY_THRMSTOR1_+V_H1-8
- removed net N$44: H1.16, H1.20, IC8.VOUT
- removed net N$52: IC6.OP, Q9.G, R28.1
- removed net N$58: C14.1, C19.1, C20.1, H2.36, IC5.VS, IC9.VDD@2, IC9.VDD@5, IC9.VREF_IN, R38.2
- new net 3V3_REG_OP_H1-16: C24.1, H1.16, H1.20, IC8.VOUT
- new net 5V_REG_OP_H1-26: C15.1, C16.1, C22.1, C23.1, C25.1, C26.1, H1.26, H1.28, IC10.RS-, IC12.ENA, IC12.VIN, IC6.VCC, IC7.VCC, IC8.VIN, R2.2, R25.2, R26.2, R3.2, R37.1
- new net N$2: H2.2, IC1.BAT, IC1.SNS, IC2.BAT, IC2.SNS, R18.2, R22.2
- new net N$45: IC6.OP, Q9.G
- new net Q6_3V3_H2-36: C14.1, H2.36, IC5.VS, R38.2
- net GNDA: now also C17.2, C18.2, C22.2, C23.2, C24.2, C25.2, C26.2, IC12.GND
- net N$18: now also C19.1, C20.1, IC12.VOUT, IC9.VDD@2, IC9.VDD@5, IC9.VREF_IN; no longer C15.1, C16.1, H1.26, H1.28, IC10.RS-, IC6.VCC, IC7.VCC, IC8.VIN, R11.2, R2.2, R25.2, R26.2, R28.2, R3.2, R37.1
- net N$33: no longer R11.1
- net N$43: now also C18.1; no longer IC1.BAT, IC1.SNS, IC2.BAT, IC2.SNS, R18.2, R22.2
- net N$47: now also C17.1
Other:
- note added: "3V3_CTL_H1-40"
- note added: "3V3_REG_OP_H1-16"
- note added: "3V3_REG_OP_H1-20"
- note added: "5V_REG_OP_H1-26"
- note added: "5V_REG_OP_H1-28"
- note added: "9V_CTL_H1-36"
- note added: "9V_REG_OP_H1-22"
- note added: "9V_REG_OP_H1-24"
- note added: "ANT_CTL_H1-38"
- note added: "BATTERY_HEATER_+V_H1-4"
- note added: "BATTERY_HEATER_-V_H1-6"
- note added: "BATTERY_THRMSTOR1_+V_H1-8"
- note added: "BATTERY_THRMSTOR2_+V_H1-12"
- note added: "PC_Q6_RX_RS232"
- note added: "POW_BATT_GND_H1-33"
- note added: "POW_BATT_V_FROM_BCR_H2-2"
- note added: "POW_BATT_V_TO_LOAD_H1-35"
- note added: "Q6_3V3_H2-36"
- note added: "Q6_3V3_H2-38"
- note added: "Q6_GPIO_10_H1-50"
- note added: "Q6_GPIO_13"
- note added: "Q6_GPIO_14"
- note added: "Q6_GPIO_15"
- note added: "Q6_I2C_SCL_1_H2-20"
- note added: "Q6_I2C_SDA_1_H2-18"
- note added: "Q6_PC_TX_RS232"
- note added: "SLR_PNL_GND_H1-30"
- note added: "SLR_PNL_GND_H1-31"
- note added: "SOLAR_PANEL_1_3_H1-29"
- note added: "SOLAR_PANEL_2_4_H1-2"
- note removed: "15V"
- note removed: "15V_CTL"
- note removed: "3.3V"
- note removed: "3.3V_CTL"
- note removed: "9V"
- note removed: "ANT_CTL"
- note removed: "ATTENNA_DEPLOYMENT_0"
- note removed: "ATTENNA_DEPLOYMENT_1"
- note removed: "BATTERY_HEATER_+V"
- note removed: "BATTERY_HEATER_-V"
- note removed: "BATTERY_THRMSTOR1_+V"
- note removed: "BATTERY_THRMSTOR2_+V"
- note removed: "EXT_PWR"
- note removed: "PC_Q6_RS232"
- note removed: "POW_BATT_GND"
- note removed: "POW_CONT_1"
- note removed: "Q6_3V3"
- note removed: "Q6_GPIO_1"
- note removed: "Q6_I2C_SCL_1"
- note removed: "Q6_I2C_SDA_1"
- note removed: "Q6_PC_RS232"
- note removed: "SLR_PNL_GND"
- note removed: "SOLAR_PANEL_1_3"
- note removed: "SOLAR_PANEL_2_4"
- moved on the sheet: C1, C10, C11, C12, C13, C14, C2, C3, C4, C5, C6, C7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
