File: EPS/eps-v1-0.sch (EAGLE design)
At the start: 84 parts, among them IC1 MIC79110, IC10 MAX4374-10UMAX, IC11 TLV70228DBV, IC2 MIC79110, IC3 LT3872, IC4 LT3872, IC5 INA291-D, IC6 NCS2202, IC7 NCS2202, IC8 TLV70233DBVR, IC9 AD7998, Q1 SI7448DP, Q2 SI7448DP, Q3 SI7448DP, Q4 SI7485DP, Q6 SI7485DP, Q8 SI7485DP, Q9 SI7448DP

Commit message: [EPS] Added and modified netnames of unused header pins and unconflicted netnames to match the wiring schematic netnames   The remaining conflicts are legitimate wired net conflicts, or grounding conflicts, and can only be resolved with redesign.
Connections:
- net N$11 renamed POW_9V
- net N$12 renamed ANTENNA_DEPLOYMENT_+V
- net N$13 renamed Q6_GPIO_15
- net N$15 renamed SOLAR_PANEL_2_4
- net N$18 renamed POW_5V
- net N$2 renamed BATTERY_THRMSTOR2_+V
- net N$22 renamed MECH_DEPLOY_SWITCH_+V
- net N$34 renamed SOLAR_PANEL_1_3
- net N$36 renamed Q6_GPIO_14
- net N$4 renamed BATTERY_HEATER_-V
- net N$41 renamed Q6_I2C_SDA_1
- net N$42 renamed Q6_I2C_SCL_1
- net N$43 renamed BATTERY_HEATER_+V
- net N$44 renamed POW_3V3
- net N$46 renamed EXTERNAL_POWER_+V
- net N$49 renamed Q6_GPIO_10
- net N$5 renamed Q6_GPIO_13
- net N$50 renamed BATTERY_THRMSTOR_+V
- new net BOTTOM_TEMP_SOLAR_PANEL-1: H2.9
- new net BOTTOM_TEMP_SOLAR_PANEL-2: H2.11
- new net BOTTOM_TEMP_SOLAR_PANEL-3: H2.13
- new net BOTTOM_TEMP_SOLAR_PANEL-4: H2.15
- new net ELEC_BAY_TEMP_1: H2.50
- new net MAX_Q6_RS232: H1.21
- new net N$1: H2.6
- new net N$106: H1.15
- new net N$108: H1.19
- new net N$11: H2.2
- new net N$110: H1.23
- new net N$112: H1.27
- new net N$117: H1.52
- new net N$118: H1.48
- new net N$120: H1.44
- new net N$122: H1.34
- new net N$13: H2.49
- new net N$15: H2.47
- new net N$17: H2.14
- new net N$2: H1.42
- new net N$22: H2.34
- new net N$27: H2.44
- new net N$4: H2.8
- new net N$491: H1.32
- new net N$5: H2.48
- new net N$6: H2.10
- new net N$654643543: H1.14
- new net N$78: H2.39
- new net N$79: H2.41
- new net N$80: H2.43
- new net N$81: H2.40
- new net N$811: H2.46
- new net N$82: H2.42
- new net N$83: H1.46
- new net N$85: H2.38
- new net N$87: H2.32
- new net N$88: H2.30
- new net N$89: H2.28
- new net N$9: H2.12
- new net N$90: H2.26
- new net N$92: H2.22
- new net N$93: H2.16
- new net N$99: H2.4
- new net POW_RADIO_3V3SYS: H2.27
- new net POW_RADIO_GND: H2.29
- new net POW_RADIO_VBATT: H2.45
- new net Q6_AIN_0: H1.39
- new net Q6_AIN_1: H1.43
- new net Q6_AOUT_0: H1.47
- new net Q6_AOUT_1: H1.51
- new net Q6_GPIO_0: H1.13
- new net Q6_GPIO_2: H2.24
- new net Q6_GPIO_6: H1.7
- new net Q6_GPIO_7: H1.9
- new net Q6_GPIO_8: H1.11
- new net Q6_MAX_RS232: H1.25
- new net Q6_RADIO_UART_RX: H1.18
- new net Q6_RADIO_UART_TX: H1.17
- new net Q6_SPI_CS0: H2.37
- new net Q6_SPI_CS1: H2.25
- new net Q6_SPI_SCLK: H2.21
- new net Q6_SPI_SDI_MISO: H2.35
- new net Q6_SPI_SDO_MOSI: H2.23
- new net THERMALGND1: H1.5
- new net TOP_TEMP_SOLAR_PANEL-1: H2.1
- new net TOP_TEMP_SOLAR_PANEL-2: H2.3
- new net TOP_TEMP_SOLAR_PANEL-3: H2.5
- new net TOP_TEMP_SOLAR_PANEL-4: H2.7
Other:
- note removed: "BOTTOM_TEMP_SOLAR_PANEL-1"
- note removed: "BOTTOM_TEMP_SOLAR_PANEL-2"
- note removed: "BOTTOM_TEMP_SOLAR_PANEL-3"
- note removed: "BOTTOM_TEMP_SOLAR_PANEL-4"
- note removed: "PC_Q6_RS232"
- note removed: "POW_RADIO_3.3V"
- note removed: "Q6_AIN_0"
- note removed: "Q6_AIN_1"
- note removed: "Q6_AOUT_0"
- note removed: "Q6_AOUT_1"
- note removed: "Q6_GPIO_6"
- note removed: "Q6_GPIO_7"
- note removed: "Q6_GPIO_8"
- note removed: "Q6_PC_RS232"
- note removed: "Q6_RADIO_UART_TX"
- note removed: "Q6_SPI_SCLK"
- note removed: "THERMALGND1"
- note removed: "TOP_TEMP_SOLAR_PANEL-1"
- note removed: "TOP_TEMP_SOLAR_PANEL-2"
- note removed: "TOP_TEMP_SOLAR_PANEL-3"
- note removed: "TOP_TEMP_SOLAR_PANEL-4"
