File: Wiring Harness/wiring-harness-complete-v1.0.sch (EAGLE design)
At the start: 24 parts, among them X10 SMA-142-0701-871/880, X11 SMA-142-0701-871/880, X12 SMA-142-0701-871/880, X13 SMA-142-0701-871/880, X14 SMA-142-0701-871/880, X15 SMA-142-0701-871/880, X16 5566-14, X17 SMA-142-0701-871/880, X8 SMA-142-0701-871/880, X9 SMA-142-0701-871/880

Commit message: Started updating wiring harness to include bottom 1u db25 wiring
Parts:
- removed X10: SMA-142-0701-871/880, con-coax:SMA-142-0701-871/880
Other:
- note added: "BOTTOM 1U"
- note added: "Bottom DB25-1"
- note added: "Bottom DB25-2"
- note added: "Note: Need find connectors for internal elec bay connections of: * battery +/- * battery thermistors * battery heating element +/-"
- note added: "Note: The JTAG connector may note be implemented. Need to check manufactured PCB"
- moved on the sheet: SV1, SV2, X11, X2, X3, X5, X6, X8
Changed lines of the file:
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@@
 <?xml version="1.0" encoding="utf-8"?>
 <!DOCTYPE eagle SYSTEM "eagle.dtd">
-<eagle version="7.3.0">
+<eagle version="7.2.0">
 <drawing>
 <settings>
@@
 <setting verticaltext="up"/>
 </settings>
-<grid distance="0.1" unitdist="inch" unit="inch" style="lines" multiple="1" display="yes" altdistance="0.01" altunitdist="inch" altunit="inch"/>
+<grid distance="0.1" unitdist="inch" unit="inch" style="lines" multiple="1" display="no" altdistance="0.01" altunitdist="inch" altunit="inch"/>
 <layers>
 <layer number="1" name="Top" color="4" fill="1" visible="no" active="no"/>
@@
 <part name="X8" library="con-coax" deviceset="SMA-" device="142-0701-871/880"/>
 <part name="X9" library="con-coax" deviceset="SMA-" device="142-0701-871/880"/>
-<part name="X10" library="con-coax" deviceset="SMA-" device="142-0701-871/880"/>
 <part name="SUPPLY11" library="supply2" deviceset="GND" device=""/>
 <part name="SUPPLY16" library="supply2" deviceset="GND" device=""/>
@@
 <wire x1="-474.98" y1="78.74" x2="-474.98" y2="284.48" width="0.1524" layer="152" style="longdash"/>
 <text x="-472.44" y="287.02" size="2.54" layer="152">TOP 1U</text>
+<text x="-170.18" y="269.24" size="1.778" layer="152">Note: Need find connectors for internal elec bay connections of:
+* battery +/-
+* battery thermistors
+* battery heating element +/-</text>
+<text x="-10.16" y="167.64" size="1.778" layer="152">Note:
+The JTAG connector may note be implemented. Need to check manufactured PCB</text>
+<wire x1="116.84" y1="-208.28" x2="360.68" y2="-208.28" width="0.1524" layer="152" style="longdash"/>
+<wire x1="116.84" y1="-208.28" x2="116.84" y2="35.56" width="0.1524" layer="152" style="longdash"/>
+<wire x1="360.68" y1="-208.28" x2="360.68" y2="35.56" width="0.1524" layer="152" style="longdash"/>
+<wire x1="116.84" y1="35.56" x2="360.68" y2="35.56" width="0.1524" layer="152" style="longdash"/>
+<text x="119.38" y="38.1" size="2.54" layer="152">BOTTOM 1U</text>
+<text x="43.18" y="-116.84" size="1.778" layer="152">Bottom DB25-1</text>
+<text x="43.18" y="-162.56" size="1.778" layer="152">Bottom DB25-2</text>
+<text x="66.04" y="-127" size="1.778" layer="95">SOLAR_PANEL_2_4</text>
 </plain>
 <instances>
@@
 <instance part="+3V12" gate="G$1" x="52.07" y="-10.16" rot="R270"/>
 <instance part="X1" gate="-1" x="-157.48" y="213.36"/>
-<instance part="X2" gate="-1" x="172.72" y="111.76"/>
-<instance part="X3" gate="-1" x="172.72" y="38.1"/>
-<instance part="X5" gate="-1" x="200.66" y="114.3"/>
-<instance part="X6" gate="-1" x="200.66" y="38.1"/>
+<instance part="X2" gate="-1" x="50.8" y="-137.16"/>
+<instance part="X3" gate="-1" x="50.8" y="-182.88"/>
+<instance part="X5" gate="-1" x="147.32" y="-137.16"/>
+<instance part="X6" gate="-1" x="147.32" y="-180.34"/>
 <instance part="X7" gate="G$1" x="-421.64" y="215.9"/>
-<instance part="X8" gate="G1" x="-160.02" y="50.8"/>
+<instance part="X8" gate="G1" x="-142.24" y="55.88"/>
 <instance part="X9" gate="G1" x="-325.12" y="154.94" rot="R180"/>
-<instance part="X10" gate="G1" x="213.36" y="-5.08" rot="R180"/>
 <instance part="SUPPLY11" gate="GND" x="-66.04" y="68.58" rot="R270"/>
 <instance part="SUPPLY16" gate="GND" x="59.69" y="68.58" rot="R90"/>
@@
 <instance part="SUPPLY28" gate="GND" x="-66.04" y="78.74" rot="R270"/>
 <instance part="SUPPLY29" gate="GND" x="58.42" y="78.74" rot="R90"/>
-<instance part="X11" gate="G1" x="-124.46" y="50.8" rot="R180"/>
+<instance part="X11" gate="G1" x="-106.68" y="55.88" rot="R180"/>
 <instance part="X12" gate="G1" x="-147.32" y="33.02"/>
 <instance part="X13" gate="G1" x="-147.32" y="12.7"/>
@@
 <instance part="X4" gate="-1" x="-325.12" y="213.36"/>
 <instance part="SUPPLY5" gate="GND" x="-337.82" y="190.5"/>
-<instance part="SV1" gate="1" x="38.1" y="-185.42"/>
-<instance part="SV2" gate="1" x="38.1" y="-154.94"/>
+<instance part="SV1" gate="1" x="-25.4" y="-180.34"/>
+<instance part="SV2" gate="1" x="-25.4" y="-139.7"/>
 </instances>
 <busses>
@@
 <wire x1="-15.24" y1="-81.28" x2="-43.18" y2="-81.28" width="0.1524" layer="91"/>
 <label x="-40.64" y="-81.28" size="1.778" layer="95"/>
+<label x="66.04" y="-124.46" size="1.778" layer="95"/>
+</segment>
+<segment>
+<wire x1="86.36" y1="-124.46" x2="58.42" y2="-124.46" width="0.1524" layer="91"/>
 </segment>
 </net>
@@
 <pinref part="H1" gate="G$1" pin="2"/>
 <wire x1="7.62" y1="-45.72" x2="38.1" y2="-45.72" width="0.1524" layer="91"/>
+</segment>
+<segment>
+<wire x1="58.42" y1="-127" x2="86.36" y2="-127" width="0.1524" layer="91"/>
 </segment>
 </net>
@@
 <wire x1="-15.24" y1="-83.82" x2="-43.18" y2="-83.82" width="0.1524" layer="91"/>
 <label x="-40.64" y="-83.82" size="1.778" layer="95"/>
+<label x="66.04" y="-134.62" size="1.778" layer="95"/>
+</segment>
+<segment>
+<wire x1="86.36" y1="-134.62" x2="58.42" y2="-134.62" width="0.1524" layer="91"/>
 </segment>
 </net>
@@
 <wire x1="7.62" y1="-81.28" x2="45.72" y2="-81.28" width="0.1524" layer="91"/>
 <label x="17.78" y="-81.28" size="1.778" layer="95"/>
+<label x="66.04" y="-137.16" size="1.778" layer="95"/>
+</segment>
+<segment>
+<wire x1="58.42" y1="-137.16" x2="86.36" y2="-137.16" width="0.1524" layer="91"/>
 </segment>
 </net>
@@
 <pinref part="X11" gate="G1" pin="1"/>
 <pinref part="X8" gate="G1" pin="1"/>
-<wire x1="-127" y1="50.8" x2="-157.48" y2="50.8" width="0.1524" layer="91"/>
-<label x="-154.94" y="50.8" size="1.778" layer="95"/>
+<wire x1="-109.22" y1="55.88" x2="-139.7" y2="55.88" width="0.1524" layer="91"/>
+<label x="-137.16" y="55.88" size="1.778" layer="95"/>
 </segment>
 <segment>
@@
 <segment>
 <pinref part="X11" gate="G1" pin="2"/>
-<wire x1="-127" y1="53.34" x2="-142.24" y2="53.34" width="0.1524" layer="91"/>
-<wire x1="-142.24" y1="53.34" x2="-142.24" y2="48.26" width="0.1524" layer="91"/>
+<wire x1="-109.22" y1="58.42" x2="-124.46" y2="58.42" width="0.1524" layer="91"/>
+<wire x1="-124.46" y1="58.42" x2="-124.46" y2="53.34" width="0.1524" layer="91"/>
 <pinref part="X8" gate="G1" pin="2"/>
-<wire x1="-142.24" y1="48.26" x2="-157.48" y2="48.26" width="0.1524" layer="91"/>
-<label x="-154.94" y="48.26" size="1.778" layer="95"/>
+<wire x1="-124.46" y1="53.34" x2="-139.7" y2="53.34" width="0.1524" layer="91"/>
+<label x="-137.16" y="53.34" size="1.778" layer="95"/>
 </segment>
 <segment>
@@
 </schematic>
 </drawing>
+<compatibility>
+<note version="6.3" minversion="6.2.2" severity="warning">
+Since Version 6.2.2 text objects can contain more than one line,
+which will not be processed correctly with this version.
+</note>
+</compatibility>
 </eagle>

Commit message: updating wiring harness as per "20131201 - Continuity Check" test
Parts:
- added J1: 22-27-2021-02, con-molex:22-27-2021-02
- added SW1, SW2, SW3: CT10-XXXX-A2, switch-coto:CT10-XXXX-A2
Connections:
- new net CONTINUITY_1: X4.12
- new net CONTINUITY_2: X4.13
- new net N$3: SW1.1, SW2.1, SW3.2
- net EXTERNAL_POWER_+V: no longer X7.2
- net EXTERNAL_POWER_GND: no longer X7.1
- net PA3_JTAG_TCK: now also X7.8; no longer X7.5
- net PA3_JTAG_TDI: no longer X7.3
- net PA3_JTAG_TDO: no longer X7.6
- net PA3_JTAG_TMS: no longer X7.4
- net PC_Q6_RS232: no longer X1.9, X4.9, X7.13
- net Q6_PC_RS232: no longer X1.8, X4.8, X7.12
- net S6_JTAG_TCK: no longer X7.10
- net S6_JTAG_TDI: no longer X7.8
- net S6_JTAG_TDO: no longer X7.11
- net S6_JTAG_TMS: no longer X7.9
- net ~PA3_JTAG_TRST: no longer X7.7
Other:
- note added: "*Note: AHRM - find connector used and correct the part #"
- note added: "*Note: Assuming Pin8(tx-) &10(rx-) are rs232 ground"
- note added: "*Note: Custom RBF assembly"
- note added: "*Todo: find actual switches used and create custom part"

Commit message: Updated Payload internal schem with notes from "20131201 - Continuity Check" Added connections to wiring harness schematic as per "20131201 - Continuity Check"
Parts:
- removed SV1, SV2: (no value), con-ml:ML16
- added U$4, U$5: M80-866XXXX, harwin:M80-866XXXX
Connections:
- removed net SLR_PNL_GND: H1.30
- new net N$18: U$5.10
- new net N$20: U$5.11
- new net N$32: U$4.5
- new net N$33: U$4.6
- new net N$34: U$4.8
- new net N$35: U$4.7
- new net N$37: U$4.14
- new net N$39: U$4.13
- new net PAYGND: U$4.9
- net +3V3: now also U$5.13
- net ANTENNA_DEPLOYMENT_+V: now also U$4.16
- net ANTENNA_DEPLOYMENT_GND: now also U$4.15
- net BOTTOM_TEMP_SOLAR_PANEL-1: now also U$5.5
- net BOTTOM_TEMP_SOLAR_PANEL-2: now also U$5.6
- net BOTTOM_TEMP_SOLAR_PANEL-3: now also U$5.7
- net BOTTOM_TEMP_SOLAR_PANEL-4: now also U$5.8
- net GND: now also U$5.14, X2.19
- net POW_5V: now also U$5.12
- net Q6_AIN_0: now also U$4.11
- net Q6_AOUT_0: now also U$4.10
- net Q6_I2C_SCL_1: now also U$5.15
- net Q6_I2C_SDA_1: now also U$5.16
- net SOLAR_PANEL_1_3: now also U$4.1, X2.4
- net SOLAR_PANEL_2_4: now also U$4.3, X2.2
- net SOLAR_PANEL_GND: now also H1.30, X2.15, X2.17
- net THERMALGND1: now also X3.14, X3.15, X3.16, X3.17, X3.18, X3.19, X3.20, X3.21, X3.22
- net TOP_TEMP_SOLAR_PANEL-1: now also U$5.1
- net TOP_TEMP_SOLAR_PANEL-2: now also U$5.2
- net TOP_TEMP_SOLAR_PANEL-3: now also U$5.3
- net TOP_TEMP_SOLAR_PANEL-4: now also U$5.4
Other:
- note added: "*Note DB25(-X) pin 9 connection unclear"
- note added: "*Note: This is the "+X" 16pin Conn"
- note added: "*Note: This is the "-X" 16pin Conn"
- note added: "Bottom DB25-1 (+X)"
- note added: "Bottom DB25-2 (-X)"
- note removed: "Bottom DB25-1"
- note removed: "Bottom DB25-2"

Commit message: added directory for eagle lbrs working on bottom 1u wiring harness according to solar panel bom and "20131201 - Continuity Check"
Parts:
- X5, X6: device con-subd:M25VB -> con-subd:M25VP
Connections:
- net +3V3: now also X2.5, X5.5
- net ANTENNA_DEPLOYMENT_+V: now also X2.13, X5.13
- net ANTENNA_DEPLOYMENT_GND: now also X2.25, X5.25
- net BOTTOM_TEMP_SOLAR_PANEL-1: now also X3.8, X6.8
- net BOTTOM_TEMP_SOLAR_PANEL-2: now also X3.4, X6.4
- net BOTTOM_TEMP_SOLAR_PANEL-3: now also X3.6, X6.6
- net BOTTOM_TEMP_SOLAR_PANEL-4: now also X3.2, X6.2
- net GND: now also X2.18, X3.24, X5.18, X5.19, X6.24
- net POW_9V: now also U$4.12, X2.6, X5.6
- net Q6_AIN_0: now also X3.11, X6.11
- net Q6_I2C_SCL_1: now also X3.10, X6.10
- net Q6_I2C_SDA_1: now also X3.23, X6.23
- net SOLAR_PANEL_1_3: now also X2.3, X5.3, X5.4
- net SOLAR_PANEL_2_4: now also X2.1, X5.1, X5.2
- net SOLAR_PANEL_GND: now also U$4.2, U$4.4, X2.14, X2.16, X5.14, X5.15, X5.16, X5.17
- net THERMALGND1: now also U$5.9, X6.14, X6.15, X6.16, X6.17, X6.18, X6.19, X6.20, X6.21, X6.22
- net TOP_TEMP_SOLAR_PANEL-1: now also X3.7, X6.7
- net TOP_TEMP_SOLAR_PANEL-2: now also X3.3, X6.3
- net TOP_TEMP_SOLAR_PANEL-3: now also X3.5, X6.5
- net TOP_TEMP_SOLAR_PANEL-4: now also X3.1, X6.1
Other:
- moved on the sheet: X2, X3, X5, X6

Commit message: - finished bottom 1u wiring harness as per "20131201 - Continuity Check"
Parts:
- added J2: 22-27-2041-04, con-molex:22-27-2041-04
- added J3: 22-05-7028-02, con-molex:22-05-7028-02
- added SL1, SL2, SL3: (no value), con-amp-quick:MA04
- added U$6, U$7, U$8, U$9: GLENAIR-171-006-6-S-6-7-18, space-concordia-power:GLENAIR-171-006-6-S-6-7-18
Connections:
- new net N$7: SL1.1, SL2.1
- new net N$8: SL1.4, SL2.4
- net GND: now also SL1.3, SL2.3, SL3.3
- net POW_9V: now also SL3.2
- net Q6_AIN_0: now also SL1.2, SL2.2
- net SOLAR_PANEL_1_3: now also U$8.3
- net SOLAR_PANEL_GND: now also U$8.2
- net THERMALGND1: now also U$8.5
- net TOP_TEMP_SOLAR_PANEL-1: now also U$6.4
Other:
- note added: "(Connect to DB25-Z+X pin01)"
- note added: "(Connect to DB25-Z+X pin02)"
- note added: "(Connect to DB25-Z+X pin03)"
- note added: "(Connect to DB25-Z+X pin04)"
- note added: "(Connect to DB25-Z+X pin14)"
- note added: "(Connect to DB25-Z+X pin15)"
- note added: "(Connect to DB25-Z+X pin16)"
- note added: "(Connect to DB25-Z+X pin17)"
- note added: "(Connect to DB25-Z-X pin01)"
- note added: "(Connect to DB25-Z-X pin02)"
- note added: "(Connect to DB25-Z-X pin03)"
- note added: "(Connect to DB25-Z-X pin04)"
- note added: "(Connect to DB25-Z-X pin05)"
- note added: "(Connect to DB25-Z-X pin06)"
- note added: "(Connect to DB25-Z-X pin07)"
- note added: "(Connect to DB25-Z-X pin08)"
- note added: "(Connect to DB25-Z-X pin14)"
- note added: "(Connect to DB25-Z-X pin15)"
- note added: "(Connect to DB25-Z-X pin16)"
- note added: "(Connect to DB25-Z-X pin17)"
- note added: "(Connect to DB25-Z-X pin18)"
- note added: "(Connect to DB25-Z-X pin19)"
- note added: "(Connect to DB25-Z-X pin20)"
- note added: "(Connect to DB25-Z-X pin21)"
- note added: "*Note ADS (ACS?) Magnetometer PCB: no connector used, direct solder to through hole"
- note added: "*Note: Payload PCB Connector - find out actual part # and create model - payload PCB apparently has 2 4pin connectors but only 2 pins of each are used?"
- note added: "*Note: Payload Thermistor - no connector used, direct solder from wiring harness"
- note added: "*Note: This is the connector for SolarPanel1"
- note added: "*Note: This is the connector for SolarPanel2"
- note added: "*Note: This is the connector for SolarPanel3"
- note added: "*Note: This is the connector for SolarPanel4"

Commit message: worked on the wiring harness:   - fixed some signals between ext payload and int payload   - added wire data.ods sheet
ran 'snap to grid' on internal payload schematic
Connections:
- net N$32 renamed G-M-OUTPUT-AMPLITUDE
- net N$33 renamed HV_OUTPUT1
- net N$34 renamed VOLTAGE_SWEEP1
- net N$35 renamed HV_OUTPUT2
- net N$37 renamed VOLTAGE_SWEEP2
- net N$39 renamed PULSE1
- removed net N$18: U$5.10
- removed net N$20: U$5.11
- removed net PAYGND: U$4.9
- new net +5V: U$5.12
- net GND: now also U$4.2, U$4.4, U$4.9, U$5.10, U$5.11, U$5.9
- net POW_5V: no longer U$5.12
- net SOLAR_PANEL_GND: no longer U$4.2, U$4.4
- net THERMALGND1: no longer U$5.9
Other:
- note added: "GND1"
- note added: "GND2"
- note added: "GND3"
- note added: "SOLAR_PANEL_GND"
- note added: "THERMALGND"

Commit message: Wiring Harness   - review and update wire data spreadsheet with Pierre-Lucas   - review and update schematic to track spreadsheet
misc
  - updated gitignore to ignore libreoffice locks
Parts:
- added D1, D2, D3, D4: 1N4004, diode:1N4004
Connections:
- new net SOLAR_PANEL_1: U$6.3
- new net SOLAR_PANEL_2: U$7.3
- new net SOLAR_PANEL_3: U$8.3
- new net SOLAR_PANEL_4: U$9.3
- net SOLAR_PANEL_1_3: no longer U$8.3
Other:
- note removed: "(Connect to DB25-Z+X pin01)"
- note removed: "(Connect to DB25-Z+X pin02)"
- note removed: "(Connect to DB25-Z+X pin03)"
- note removed: "(Connect to DB25-Z+X pin04)"
Changed lines of the file:
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@@
 <setting verticaltext="up"/>
 </settings>
-<grid distance="1.27" unitdist="mm" unit="mm" style="dots" multiple="1" display="yes" altdistance="0.127" altunitdist="mm" altunit="mm"/>
+<grid distance="1.27" unitdist="mm" unit="mm" style="lines" multiple="1" display="no" altdistance="0.254" altunitdist="mm" altunit="mm"/>
 <layers>
 <layer number="1" name="Top" color="4" fill="1" visible="no" active="no"/>
@@
 <layer number="97" name="Info" color="7" fill="1" visible="yes" active="yes"/>
 <layer number="98" name="Guide" color="6" fill="1" visible="yes" active="yes"/>
+<layer number="99" name="SpiceOrder" color="5" fill="1" visible="yes" active="yes"/>
 <layer number="100" name="Muster" color="7" fill="1" visible="no" active="no"/>
 <layer number="101" name="Patch_Top" color="12" fill="4" visible="yes" active="yes"/>
@@
 <part name="+3V1" library="supply1" deviceset="+3V3" device=""/>
 <part name="P+1" library="supply1" deviceset="+5V" device=""/>
+<part name="D1" library="diode" deviceset="1N4004" device=""/>
+<part name="D2" library="diode" deviceset="1N4004" device=""/>
+<part name="D3" library="diode" deviceset="1N4004" device=""/>
+<part name="D4" library="diode" deviceset="1N4004" device=""/>
 </parts>
 <sheets>
@@
 <text x="147.32" y="17.78" size="1.778" layer="152">(Connect to DB25-Z-X pin20)</text>
 <text x="147.32" y="-12.7" size="1.778" layer="152">(Connect to DB25-Z-X pin21)</text>
-<text x="147.32" y="2.54" size="1.778" layer="152">(Connect to DB25-Z+X pin04)</text>
 <text x="147.32" y="10.16" size="1.778" layer="152">(Connect to DB25-Z+X pin17)</text>
 <text x="147.32" y="-5.08" size="1.778" layer="152">(Connect to DB25-Z-X pin07)</text>
@@
 <text x="204.47" y="17.78" size="1.778" layer="152">(Connect to DB25-Z-X pin03)</text>
 <text x="204.47" y="-12.7" size="1.778" layer="152">(Connect to DB25-Z-X pin19)</text>
-<text x="204.47" y="2.54" size="1.778" layer="152">(Connect to DB25-Z+X pin02)</text>
 <text x="204.47" y="10.16" size="1.778" layer="152">(Connect to DB25-Z+X pin16)</text>
 <text x="204.47" y="-5.08" size="1.778" layer="152">(Connect to DB25-Z-X pin18)</text>
@@
 <text x="261.62" y="17.78" size="1.778" layer="152">(Connect to DB25-Z-X pin05)</text>
 <text x="261.62" y="-12.7" size="1.778" layer="152">(Connect to DB25-Z-X pin17)</text>
-<text x="261.62" y="2.54" size="1.778" layer="152">(Connect to DB25-Z+X pin03)</text>
 <text x="261.62" y="10.16" size="1.778" layer="152">(Connect to DB25-Z+X pin15)</text>
 <text x="261.62" y="-5.08" size="1.778" layer="152">(Connect to DB25-Z-X pin16)</text>
@@
 <text x="320.04" y="17.78" size="1.778" layer="152">(Connect to DB25-Z-X pin01)</text>
 <text x="320.04" y="-12.7" size="1.778" layer="152">(Connect to DB25-Z-X pin02)</text>
-<text x="320.04" y="2.54" size="1.778" layer="152">(Connect to DB25-Z+X pin01)</text>
 <text x="320.04" y="10.16" size="1.778" layer="152">(Connect to DB25-Z+X pin14)</text>
 <text x="320.04" y="-5.08" size="1.778" layer="152">(Connect to DB25-Z-X pin14)</text>
@@
 <instance part="+3V1" gate="G$1" x="-27.94" y="-139.7"/>
 <instance part="P+1" gate="1" x="-22.86" y="-142.24"/>
+<instance part="D1" gate="1" x="157.48" y="-30.48"/>
+<instance part="D2" gate="1" x="218.44" y="-30.48"/>
+<instance part="D3" gate="1" x="274.32" y="-30.48"/>
+<instance part="D4" gate="1" x="327.66" y="-30.48"/>
 </instances>
 <busses>
@@
 </segment>
 <segment>
-<wire x1="154.94" y1="5.08" x2="144.78" y2="5.08" width="0.1524" layer="91"/>
-<label x="147.32" y="5.08" size="1.778" layer="95"/>
-</segment>
-<segment>
-<wire x1="269.24" y1="5.08" x2="259.08" y2="5.08" width="0.1524" layer="91"/>
-<label x="261.62" y="5.08" size="1.778" layer="95"/>
-<pinref part="U$8" gate="G$1" pin="3"/>
+<wire x1="170.18" y1="-30.48" x2="160.02" y2="-30.48" width="0.1524" layer="91"/>
+<wire x1="170.18" y1="-30.48" x2="160.02" y2="-30.48" width="0.1524" layer="91"/>
+<label x="170.18" y="-30.48" size="1.778" layer="95"/>
+</segment>
+<segment>
+<wire x1="287.02" y1="-30.48" x2="276.86" y2="-30.48" width="0.1524" layer="91"/>
+<label x="287.02" y="-30.48" size="1.778" layer="95"/>
 </segment>
 </net>
@@
 </segment>
 <segment>
-<wire x1="201.93" y1="5.08" x2="212.09" y2="5.08" width="0.1524" layer="91"/>
-<label x="204.47" y="5.08" size="1.778" layer="95"/>
-</segment>
-<segment>
-<wire x1="317.5" y1="5.08" x2="327.66" y2="5.08" width="0.1524" layer="91"/>
-<label x="320.04" y="5.08" size="1.778" layer="95"/>
+<wire x1="220.98" y1="-30.48" x2="228.6" y2="-30.48" width="0.1524" layer="91"/>
+<wire x1="220.98" y1="-30.48" x2="228.6" y2="-30.48" width="0.1524" layer="91"/>
+<label x="228.6" y="-30.48" size="1.778" layer="95"/>
+</segment>
+<segment>
+<wire x1="330.2" y1="-30.48" x2="337.82" y2="-30.48" width="0.1524" layer="91"/>
+<label x="337.82" y="-30.48" size="1.778" layer="95"/>
 </segment>
 </net>
@@
 </segment>
 </net>
+<net name="SOLAR_PANEL_1" class="0">
+<segment>
+<pinref part="U$6" gate="G$1" pin="3"/>
+<wire x1="144.78" y1="5.08" x2="154.94" y2="5.08" width="0.1524" layer="91"/>
+<label x="147.32" y="5.08" size="1.778" layer="95"/>
+</segment>
+<segment>
+<wire x1="144.78" y1="-30.48" x2="154.94" y2="-30.48" width="0.1524" layer="91"/>
+</segment>
+</net>
+<net name="SOLAR_PANEL_2" class="0">
+<segment>
+<pinref part="U$7" gate="G$1" pin="3"/>
+<wire x1="201.93" y1="5.08" x2="212.09" y2="5.08" width="0.1524" layer="91"/>
+<label x="204.47" y="5.08" size="1.778" layer="95"/>
+<wire x1="201.93" y1="5.08" x2="212.09" y2="5.08" width="0.1524" layer="91"/>
+</segment>
+<segment>
+<wire x1="205.74" y1="-30.48" x2="215.9" y2="-30.48" width="0.1524" layer="91"/>
+</segment>
+</net>
+<net name="SOLAR_PANEL_3" class="0">
+<segment>
+<pinref part="U$8" gate="G$1" pin="3"/>
+<wire x1="259.08" y1="5.08" x2="269.24" y2="5.08" width="0.1524" layer="91"/>
+<label x="261.62" y="5.08" size="1.778" layer="95"/>
+</segment>
+<segment>
+<wire x1="261.62" y1="-30.48" x2="271.78" y2="-30.48" width="0.1524" layer="91"/>
+</segment>
+</net>
+<net name="SOLAR_PANEL_4" class="0">
+<segment>
+<pinref part="U$9" gate="G$1" pin="3"/>
+<wire x1="317.5" y1="5.08" x2="327.66" y2="5.08" width="0.1524" layer="91"/>
+<label x="320.04" y="5.08" size="1.778" layer="95"/>
+</segment>
+<segment>
+<wire x1="314.96" y1="-30.48" x2="325.12" y2="-30.48" width="0.1524" layer="91"/>
+</segment>
+</net>
