File: Wiring Harness/wiring-harness-complete-v1.0.sch (EAGLE design)
At the start: 24 parts, among them X10 SMA-142-0701-871/880, X11 SMA-142-0701-871/880, X12 SMA-142-0701-871/880, X13 SMA-142-0701-871/880, X14 SMA-142-0701-871/880, X15 SMA-142-0701-871/880, X16 5566-14, X17 SMA-142-0701-871/880, X8 SMA-142-0701-871/880, X9 SMA-142-0701-871/880

Commit message: merged in updates from cs1dev branch for:   wiring harness   acs and diplexer boms   lbr (eagle libraries)
Parts:
- removed SV1, SV2: (no value), con-ml:ML16
- removed X10: SMA-142-0701-871/880, con-coax:SMA-142-0701-871/880
- added J1: 22-27-2021-02, con-molex:22-27-2021-02
- added J2: 22-27-2041-04, con-molex:22-27-2041-04
- added J3: 22-05-7028-02, con-molex:22-05-7028-02
- added SL1, SL2, SL3: (no value), con-amp-quick:MA04
- added SW1, SW2, SW3: CT10-XXXX-A2, switch-coto:CT10-XXXX-A2
- added U$4, U$5: M80-866XXXX, harwin:M80-866XXXX
- added U$6, U$7, U$8, U$9: GLENAIR-171-006-6-S-6-7-18, space-concordia-power:GLENAIR-171-006-6-S-6-7-18
- X5, X6: device con-subd:M25VB -> con-subd:M25VP
Connections:
- removed net SLR_PNL_GND: H1.30
- new net CONTINUITY_1: X4.12
- new net CONTINUITY_2: X4.13
- new net N$18: U$5.10
- new net N$20: U$5.11
- new net N$3: SW1.1, SW2.1, SW3.2
- new net N$32: U$4.5
- new net N$33: U$4.6
- new net N$34: U$4.8
- new net N$35: U$4.7
- new net N$37: U$4.14
- new net N$39: U$4.13
- new net N$7: SL1.1, SL2.1
- new net N$8: SL1.4, SL2.4
- new net PAYGND: U$4.9
- net +3V3: now also U$5.13, X2.5, X5.5
- net ANTENNA_DEPLOYMENT_+V: now also U$4.16, X2.13, X5.13
- net ANTENNA_DEPLOYMENT_GND: now also U$4.15, X2.25, X5.25
- net BOTTOM_TEMP_SOLAR_PANEL-1: now also U$5.5, X3.8, X6.8
- net BOTTOM_TEMP_SOLAR_PANEL-2: now also U$5.6, X3.4, X6.4
- net BOTTOM_TEMP_SOLAR_PANEL-3: now also U$5.7, X3.6, X6.6
- net BOTTOM_TEMP_SOLAR_PANEL-4: now also U$5.8, X3.2, X6.2
- net EXTERNAL_POWER_+V: no longer X7.2
- net EXTERNAL_POWER_GND: no longer X7.1
- net GND: now also SL1.3, SL2.3, SL3.3, U$5.14, X2.18, X2.19, X3.24, X5.18, X5.19, X6.24
- net PA3_JTAG_TCK: now also X7.8; no longer X7.5
- net PA3_JTAG_TDI: no longer X7.3
- net PA3_JTAG_TDO: no longer X7.6
- net PA3_JTAG_TMS: no longer X7.4
- net PC_Q6_RS232: no longer X1.9, X4.9, X7.13
- net POW_5V: now also U$5.12
- net POW_9V: now also SL3.2, U$4.12, X2.6, X5.6
- net Q6_AIN_0: now also SL1.2, SL2.2, U$4.11, X3.11, X6.11
- net Q6_AOUT_0: now also U$4.10
- net Q6_I2C_SCL_1: now also U$5.15, X3.10, X6.10
- net Q6_I2C_SDA_1: now also U$5.16, X3.23, X6.23
- net Q6_PC_RS232: no longer X1.8, X4.8, X7.12
- net S6_JTAG_TCK: no longer X7.10
- net S6_JTAG_TDI: no longer X7.8
- net S6_JTAG_TDO: no longer X7.11
- net S6_JTAG_TMS: no longer X7.9
- net SOLAR_PANEL_1_3: now also U$4.1, U$8.3, X2.3, X2.4, X5.3, X5.4
- net SOLAR_PANEL_2_4: now also U$4.3, X2.1, X2.2, X5.1, X5.2
- net SOLAR_PANEL_GND: now also H1.30, U$4.2, U$4.4, U$8.2, X2.14, X2.15, X2.16, X2.17, X5.14, X5.15, X5.16, X5.17
- net THERMALGND1: now also U$5.9, U$8.5, X3.14, X3.15, X3.16, X3.17, X3.18, X3.19, X3.20, X3.21, X3.22, X6.14, X6.15, X6.16, X6.17, X6.18, X6.19, X6.20, X6.21, X6.22
- net TOP_TEMP_SOLAR_PANEL-1: now also U$5.1, U$6.4, X3.7, X6.7
- net TOP_TEMP_SOLAR_PANEL-2: now also U$5.2, X3.3, X6.3
- net TOP_TEMP_SOLAR_PANEL-3: now also U$5.3, X3.5, X6.5
- net TOP_TEMP_SOLAR_PANEL-4: now also U$5.4, X3.1, X6.1
- net ~PA3_JTAG_TRST: no longer X7.7
Other:
- note added: "(Connect to DB25-Z+X pin01)"
- note added: "(Connect to DB25-Z+X pin02)"
- note added: "(Connect to DB25-Z+X pin03)"
- note added: "(Connect to DB25-Z+X pin04)"
- note added: "(Connect to DB25-Z+X pin14)"
- note added: "(Connect to DB25-Z+X pin15)"
- note added: "(Connect to DB25-Z+X pin16)"
- note added: "(Connect to DB25-Z+X pin17)"
- note added: "(Connect to DB25-Z-X pin01)"
- note added: "(Connect to DB25-Z-X pin02)"
- note added: "(Connect to DB25-Z-X pin03)"
- note added: "(Connect to DB25-Z-X pin04)"
- note added: "(Connect to DB25-Z-X pin05)"
- note added: "(Connect to DB25-Z-X pin06)"
- note added: "(Connect to DB25-Z-X pin07)"
- note added: "(Connect to DB25-Z-X pin08)"
- note added: "(Connect to DB25-Z-X pin14)"
- note added: "(Connect to DB25-Z-X pin15)"
- note added: "(Connect to DB25-Z-X pin16)"
- note added: "(Connect to DB25-Z-X pin17)"
- note added: "(Connect to DB25-Z-X pin18)"
- note added: "(Connect to DB25-Z-X pin19)"
- note added: "(Connect to DB25-Z-X pin20)"
- note added: "(Connect to DB25-Z-X pin21)"
- note added: "*Note ADS (ACS?) Magnetometer PCB: no connector used, direct solder to through hole"
- note added: "*Note DB25(-X) pin 9 connection unclear"
- note added: "*Note: AHRM - find connector used and correct the part #"
- note added: "*Note: Assuming Pin8(tx-) &10(rx-) are rs232 ground"
- note added: "*Note: Custom RBF assembly"
- note added: "*Note: Payload PCB Connector - find out actual part # and create model - payload PCB apparently has 2 4pin connectors but only 2 pins of each are used?"
- note added: "*Note: Payload Thermistor - no connector used, direct solder from wiring harness"
- note added: "*Note: This is the "+X" 16pin Conn"
- note added: "*Note: This is the "-X" 16pin Conn"
- note added: "*Note: This is the connector for SolarPanel1"
- note added: "*Note: This is the connector for SolarPanel2"
- note added: "*Note: This is the connector for SolarPanel3"
- note added: "*Note: This is the connector for SolarPanel4"
- note added: "*Todo: find actual switches used and create custom part"
- note added: "BOTTOM 1U"
- note added: "Bottom DB25-1 (+X)"
- note added: "Bottom DB25-2 (-X)"
- note added: "Note: Need find connectors for internal elec bay connections of: * battery +/- * battery thermistors * battery heating element +/-"
- note added: "Note: The JTAG connector may note be implemented. Need to check manufactured PCB"
- moved on the sheet: X11, X2, X3, X5, X6, X8

Commit message: CDH updates   - renamed H1 <-> H2 headers to match others schematics   - deleted misleading 'Q6_GPIO_10' label
Wiring harness updates
  - deleted misleading 'Q6_GPIO_10' label
Other:
- note removed: "Q6_GPIO_10"
Changed lines of the file:
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@@
 <?xml version="1.0" encoding="utf-8"?>
 <!DOCTYPE eagle SYSTEM "eagle.dtd">
-<eagle version="7.3.0">
+<eagle version="7.2.0">
 <drawing>
 <settings>
@@
 <setting verticaltext="up"/>
 </settings>
-<grid distance="1.27" unitdist="mm" unit="mm" style="lines" multiple="1" display="yes" altdistance="0.01" altunitdist="inch" altunit="mm"/>
+<grid distance="0.1" unitdist="inch" unit="inch" style="lines" multiple="1" display="no" altdistance="0.01" altunitdist="inch" altunit="inch"/>
 <layers>
 <layer number="1" name="Top" color="4" fill="1" visible="no" active="no"/>
@@
 <text x="17.78" y="-45.72" size="1.778" layer="95">SOLAR_PANEL_2_4</text>
 <text x="35.46" y="-93.59" size="1.778" layer="95">3V3_CTL</text>
-<text x="27.94" y="-106.68" size="1.778" layer="95">Q6_GPIO_10</text>
 <text x="35.56" y="124.46" size="1.778" layer="95">Q6_AOUT_0</text>
 <text x="35.56" y="121.92" size="1.778" layer="95">Q6_AOUT_1</text>

Commit message: [Wiring Harness] matched connector type and nets for ACS <-> wiring-harness
[MISC] converted the start of schematic convention doc to .MD
Parts:
- removed J2: 22-27-2041-04, con-molex:22-27-2041-04
- added J10: 22-27-2021-02, con-molex:22-27-2021-02
- J1: value 22-27-2021-02 -> M80-879; device con-molex:22-27-2021-02 -> harwin:M80-879
Connections:
- net +3V3: now also J1.2
- net GND: now also J1.1
- net Q6_I2C_SCL_1: now also J1.4
- net Q6_I2C_SDA_1: now also J1.3
Changed lines of the file:
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@@
 <setting verticaltext="up"/>
 </settings>
-<grid distance="0.1" unitdist="inch" unit="inch" style="lines" multiple="1" display="no" altdistance="0.01" altunitdist="inch" altunit="inch"/>
+<grid distance="1.27" unitdist="mm" unit="mm" style="lines" multiple="1" display="no" altdistance="0.254" altunitdist="mm" altunit="mm"/>
 <layers>
 <layer number="1" name="Top" color="4" fill="1" visible="no" active="no"/>
@@
 <part name="SW2" library="switch-coto" deviceset="CT10-XXXX-" device="A2"/>
 <part name="SW3" library="switch-coto" deviceset="CT10-XXXX-" device="A2"/>
-<part name="J1" library="con-molex" deviceset="22-?-02" device="27-2021"/>
+<part name="J10" library="con-molex" deviceset="22-?-02" device="27-2021"/>
 <part name="U$4" library="harwin" deviceset="M80-866XXXX" device=""/>
 <part name="U$5" library="harwin" deviceset="M80-866XXXX" device=""/>
@@
 <part name="U$8" library="space-concordia-power" deviceset="GLENAIR-171-006-6-S-6-7-18" device=""/>
 <part name="U$9" library="space-concordia-power" deviceset="GLENAIR-171-006-6-S-6-7-18" device=""/>
-<part name="J2" library="con-molex" deviceset="22-?-04" device="27-2041"/>
 <part name="J3" library="con-molex" deviceset="22-?-02" device="05-7028"/>
 <part name="SL1" library="con-amp-quick" deviceset="MA04" device=""/>
 <part name="SL2" library="con-amp-quick" deviceset="MA04" device=""/>
 <part name="SL3" library="con-amp-quick" deviceset="MA04" device=""/>
+<part name="J1" library="harwin" deviceset="M80-879" device="" value=""/>
 </parts>
 <sheets>
@@
 <instance part="SW2" gate="G$1" x="-363.22" y="254"/>
 <instance part="SW3" gate="G$1" x="-386.08" y="259.08"/>
-<instance part="J1" gate="-1" x="322.58" y="-172.72"/>
-<instance part="J1" gate="-2" x="322.58" y="-177.8"/>
+<instance part="J10" gate="-1" x="322.58" y="-172.72"/>
+<instance part="J10" gate="-2" x="322.58" y="-177.8"/>
 <instance part="U$4" gate="G$1" x="-73.66" y="-185.42"/>
 <instance part="U$5" gate="G$1" x="-73.66" y="-147.32"/>
@@
 <attribute name="NAME" x="304.8" y="0" size="1.778" layer="95" rot="R180"/>
 </instance>
-<instance part="J2" gate="-1" x="302.26" y="-59.69"/>
-<instance part="J2" gate="-2" x="302.26" y="-64.77"/>
-<instance part="J2" gate="-3" x="302.26" y="-69.85"/>
-<instance part="J2" gate="-4" x="302.26" y="-74.93"/>
 <instance part="J3" gate="-1" x="287.02" y="-142.24"/>
 <instance part="J3" gate="-2" x="287.02" y="-147.32"/>
@@
 <instance part="SL2" gate="G$1" x="287.02" y="-115.57" rot="R180"/>
 <instance part="SL3" gate="G$1" x="287.02" y="-99.06" rot="R180"/>
+<instance part="J1" gate="G$1" x="304.8" y="-66.04"/>
 </instances>
 <busses>
@@
 </segment>
 <segment>
-<wire x1="284.48" y1="-74.93" x2="299.72" y2="-74.93" width="0.1524" layer="91"/>
-<label x="284.48" y="-74.93" size="1.778" layer="95"/>
+<wire x1="325.12" y1="-58.42" x2="317.5" y2="-58.42" width="0.1524" layer="91"/>
+<label x="316.23" y="-60.96" size="1.778" layer="95"/>
+<pinref part="J1" gate="G$1" pin="1"/>
 </segment>
 <segment>
@@
 </segment>
 <segment>
-<wire x1="299.72" y1="-69.85" x2="284.48" y2="-69.85" width="0.1524" layer="91"/>
-<label x="284.48" y="-69.85" size="1.778" layer="95"/>
+<wire x1="317.5" y1="-63.5" x2="325.12" y2="-63.5" width="0.1524" layer="91"/>
+<label x="314.96" y="-66.04" size="1.778" layer="95"/>
+<pinref part="J1" gate="G$1" pin="2"/>
 </segment>
 </net>
@@
 </segment>
 <segment>
-<wire x1="284.48" y1="-64.77" x2="299.72" y2="-64.77" width="0.1524" layer="91"/>
-<label x="276.86" y="-64.77" size="1.778" layer="95"/>
+<wire x1="317.5" y1="-68.58" x2="325.12" y2="-68.58" width="0.1524" layer="91"/>
+<label x="314.96" y="-71.12" size="1.778" layer="95"/>
+<pinref part="J1" gate="G$1" pin="3"/>
 </segment>
 </net>
@@
 </segment>
 <segment>
-<wire x1="284.48" y1="-59.69" x2="299.72" y2="-59.69" width="0.1524" layer="91"/>
-<label x="276.86" y="-59.69" size="1.778" layer="95"/>
-</segment>
-</net>
+<wire x1="317.5" y1="-73.66" x2="325.12" y2="-73.66" width="0.1524" layer="91"/>
+<label x="314.96" y="-76.2" size="1.778" layer="95"/>
+<pinref part="J1" gate="G$1" pin="4"/>
+</segment>
+</net>

Commit message: [CDH] renamed connectors to 'J#' in sync with wiring harness [diplexer-rcl.lbr] copied rcl.lbr and created an inductor with SMD package L01005(imperial) [DIPLEXER] renamed sma connectors to 'J#' in sync with wiring harness    changed part symbols of C6 C7 C8 C9 C10 to L6 L7 L8 L9 L10 [space-concordia-power-lbr] updated 'GLENAIR-171-006-6-S-6-7-18' to have a valid prefix [Payload-Internal-Aux] renamed connectors to 'J#' in sync with wiring harness [wiring-harness] renamed all known connectors to 'J#' in sync with wiring harness
Parts:
- removed U$3: M80-5000000M1-10-331-00-000, harwin:M80-5000000M1-10-331-00-000
- removed X11, X12, X13, X14, X15, X8: SMA-142-0701-871/880, con-coax:SMA-142-0701-871/880
- added J11, J12, J15, J16, J17: SMA-142-0701-871/880, con-coax:SMA-142-0701-871/880
- added J50: 22-27-2021-02, con-molex:22-27-2021-02
- added J53: 22-05-7028-02, con-molex:22-05-7028-02
- J10: value 22-27-2021-02 -> SMA-142-0701-871/880; device con-molex:22-27-2021-02 -> con-coax:SMA-142-0701-871/880
- J3: value 22-05-7028-02 -> M80-5000000M1-10-331-00-000; device con-molex:22-05-7028-02 -> harwin:M80-5000000M1-10-331-00-000
- renumbered U$1 to J4, U$2 to J2, U$4 to J31, U$5 to J30, U$6 to J20, U$7 to J21, U$8 to J22, U$9 to J23, X1 to J40, X17 to J19, X2 to J41, X3 to J42, X4 to J43, X5 to J45, X6 to J46, X7 to J44, X9 to J18
Connections:
- net DIPLEX_TO_ANT_GND: now also J12.2, J17.2; no longer X11.2, X8.2
- net DIPLEX_TO_ANT_SIG: now also J12.1, J17.1; no longer X11.1, X8.1
- net EXTERNAL_POWER_+V: now also J3.X4; no longer U$3.X4
- net EXTERNAL_POWER_GND: now also J3.X3; no longer U$3.X3
- net HE100_RX_TO_DIPLEX_GND: now also J10.2, J16.2; no longer X13.2, X15.2
- net HE100_RX_TO_DIPLEX_SIG: now also J10.1, J16.1; no longer X13.1, X15.1
- net HE100_TX_TO_DIPLEX_GND: now also J11.2, J15.2; no longer X12.2, X14.2
- net HE100_TX_TO_DIPLEX_SIG: now also J11.1, J15.1; no longer X12.1, X14.1
- net POW_BATT_GND: now also J3.X1; no longer U$3.X1
- net POW_BATT_VOUT: now also J3.X2; no longer U$3.X2
Other:
- note added: "DIPLEXER"
- note added: "HE100"

Commit message: Fixed all the trivial wiring issues for the CDH, Diplexer, EPS and wiring harness schematics
Parts:
- J10, J11, J12, J15, J16, J17: value SMA-142-0701-871/880 -> SMA-142-0701-801/806; device con-coax:SMA-142-0701-871/880 -> con-coax:SMA-142-0701-801/806
Connections:
- net BATTERY_THRMSTOR_+V renamed BATTERY_THRMSTOR1_+V
- net POW_RADIO_3.3V renamed POW_RADIO_3V3
- net POW_RADIO_3.3VSYS renamed POW_RADIO_3V3_SYS
- removed net EXTERNAL_POWER_+V: H2.52, J3.X4, J40.5, J43.5
- removed net Q6_AOUT_2: J4.C4
- removed net Q6_AOUT_3: J4.C6
- new net EXTERNAL_POWER_V+: H2.52, J3.X3, J40.5, J43.5
- net EXTERNAL_POWER_GND: now also J3.X4; no longer J3.X3
- net PA3_PC_RS232: no longer H1.25
- net PC_PA3_RS232: no longer H1.21
- net PC_Q6_RS232: now also H1.21
- net Q6_AOUT_0: now also J4.C4
- net Q6_AOUT_1: now also J4.C6
- net Q6_PC_RS232: now also H1.25
Other:
- moved on the sheet: J12, J17

Commit message: [CDH] updated trivial mismatches between connector netnames [EPS] updated trivial mismatches between connector netnames [PAYLOAD] updated trivial mismatches between connector netnames [WIRING] updated trivial mismatches between connector netnames
Connections:
- removed net N$84: H1.50
- net Q6_GPIO_10: now also H1.50
Changed lines of the file:
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@@
 <label x="35.56" y="109.22" size="1.778" layer="95"/>
+</segment>
+<segment>
+<pinref part="H1" gate="G$1" pin="50"/>
+<wire x1="7.62" y1="-106.68" x2="46.99" y2="-106.68" width="0.1524" layer="91"/>
+<label x="17.78" y="-106.68" size="1.778" layer="95"/>
 </segment>
 </net>
@@
 </segment>
 </net>
-<net name="N$84" class="0">
-<segment>
-<pinref part="H1" gate="G$1" pin="50"/>
-<wire x1="7.62" y1="-106.68" x2="46.99" y2="-106.68" width="0.1524" layer="91"/>
-<label x="17.78" y="-106.68" size="1.778" layer="95"/>
-</segment>
-</net>

Commit message: Revert "Fixed all the trivial wiring issues for the CDH, Diplexer, EPS and wiring harness schematics"
This reverts commits
  6713d85a6277b26f983fd7a52d0f95a7f9e4e046.
  086194ae58682b6763f31692a26cd4dac33df983
  82b42737f0fe6cd82dfea4a4ae7507beb01cc7b8

This revert is required because changing/connecting net names in eagle will automatically modify or destroy PCB traces associated with those netnames.
Updating the schematics and PCBs will need to be redone carefully to ensure no traces are destroyed.

	modified:   CDH-V3.7/CDH-v3.7.brd
	modified:   CDH-V3.7/CDH-v3.7.sch
	modified:   Diplexer/diplexer_v4rev0-schematic.sch
	modified:   EPS/eps-v1-0.brd
	modified:   EPS/eps-v1-0.sch
	modified:   Payload Internal - Auxiliary/Payload v2.1.brd
	modified:   Payload Internal - Auxiliary/Payload v2.1.sch
	modified:   Wiring Harness/wiring-harness-complete-v1.0.sch
Parts:
- J10, J11, J12, J15, J16, J17: value SMA-142-0701-801/806 -> SMA-142-0701-871/880; device con-coax:SMA-142-0701-801/806 -> con-coax:SMA-142-0701-871/880
Connections:
- net BATTERY_THRMSTOR1_+V renamed BATTERY_THRMSTOR_+V
- net POW_RADIO_3V3 renamed POW_RADIO_3.3V
- net POW_RADIO_3V3_SYS renamed POW_RADIO_3.3VSYS
- removed net EXTERNAL_POWER_V+: H2.52, J3.X3, J40.5, J43.5
- new net EXTERNAL_POWER_+V: H2.52, J3.X4, J40.5, J43.5
- new net N$84: H1.50
- new net Q6_AOUT_2: J4.C4
- new net Q6_AOUT_3: J4.C6
- net EXTERNAL_POWER_GND: now also J3.X3; no longer J3.X4
- net PA3_PC_RS232: now also H1.25
- net PC_PA3_RS232: now also H1.21
- net PC_Q6_RS232: no longer H1.21
- net Q6_AOUT_0: no longer J4.C4
- net Q6_AOUT_1: no longer J4.C6
- net Q6_GPIO_10: no longer H1.50
- net Q6_PC_RS232: no longer H1.25
Other:
- moved on the sheet: J12, J17
