File: ACS/ACS_PCB.brd (EAGLE design)
At the start: 93.7 x 37.8 mm, 7 parts, among them U1 HMC5883LSMD

Commit message: [Wiring Harness] matched connector type and nets for ACS <-> wiring-harness
[MISC] converted the start of schematic convention doc to .MD
Parts:
- renumbered JP1 to J1
Connections:
- net SCL renamed Q6_I2C_SCL_1
- net SDA renamed Q6_I2C_SDA_1
- net VCC renamed +3V3
Changed lines of the file:
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@@
 <?xml version="1.0" encoding="utf-8"?>
 <!DOCTYPE eagle SYSTEM "eagle.dtd">
-<eagle version="6.2">
+<eagle version="7.2.0">
 <drawing>
 <settings>
@@
 </class>
 </classes>
-<designrules>
+<designrules name="default">
 <description language="en">&lt;b&gt;EAGLE Design Rules&lt;/b&gt;
 &lt;p&gt;
@@
 <pass name="Default">
 <param name="RoutingGrid" value="50mil"/>
+<param name="AutoGrid" value="1"/>
+<param name="Efforts" value="0"/>
+<param name="TopRouterVariant" value="1"/>
 <param name="tpViaShape" value="round"/>
 <param name="PrefDir.1" value="|"/>
@@
 <element name="R1" library="SparkFun" package="0402-RES" value="DNP" x="45.635" y="19.49" rot="R90"/>
 <element name="R2" library="SparkFun" package="0402-RES" value="DNP" x="46.905" y="19.49" rot="R90"/>
-<element name="JP1" library="harwin" package="M80-879" value="" x="10.855" y="19.1" rot="R270"/>
+<element name="J1" library="harwin" package="M80-879" value="" x="10.855" y="19.1" rot="R270"/>
 </elements>
 <signals>
-<signal name="VCC">
+<signal name="+3V3">
 <contactref element="U1" pad="4"/>
 <contactref element="U1" pad="13"/>
@@
 <contactref element="R2" pad="2"/>
 <contactref element="C1" pad="1"/>
-<contactref element="JP1" pad="2"/>
+<contactref element="J1" pad="2"/>
 <wire x1="45.635" y1="20.14" x2="46.905" y2="20.14" width="0.254" layer="1"/>
 <wire x1="45.635" y1="20.14" x2="45.62" y2="20.125" width="0.254" layer="1"/>
@@
 <wire x1="45.595" y1="20.1" x2="45.635" y2="20.14" width="0.254" layer="1"/>
 </signal>
-<signal name="SCL">
+<signal name="Q6_I2C_SCL_1">
 <contactref element="U1" pad="1"/>
 <contactref element="R1" pad="1"/>
-<contactref element="JP1" pad="4"/>
+<contactref element="J1" pad="4"/>
 <wire x1="49.965" y1="18.12" x2="49.94" y2="13.74" width="0.254" layer="1"/>
 <wire x1="49.94" y1="13.74" x2="49.325" y2="13.15" width="0.254" layer="1"/>
@@
 <wire x1="45.5" y1="13.825" x2="45.675" y2="14" width="0.254" layer="1"/>
 </signal>
-<signal name="SDA">
+<signal name="Q6_I2C_SDA_1">
 <contactref element="U1" pad="16"/>
 <contactref element="R2" pad="1"/>
-<contactref element="JP1" pad="3"/>
+<contactref element="J1" pad="3"/>
 <wire x1="46.905" y1="18.84" x2="48.225" y2="18.84" width="0.254" layer="1"/>
 <wire x1="48.225" y1="18.84" x2="48.46" y2="18.84" width="0.254" layer="1"/>
@@
 </signal>
 <signal name="GND">
-<contactref element="JP1" pad="1"/>
+<contactref element="J1" pad="1"/>
 <contactref element="C3" pad="2"/>
 <contactref element="U1" pad="9"/>
