File: ACS/ACS_PCB.sch (EAGLE design)
At the start: 7 parts, among them U1 HMC5883LSMD

Commit message: [Wiring Harness] matched connector type and nets for ACS <-> wiring-harness
[MISC] converted the start of schematic convention doc to .MD
Parts:
- renumbered JP1 to J1
Connections:
- net SCL renamed Q6_I2C_SCL_1
- net SDA renamed Q6_I2C_SDA_1
- net VCC renamed +3V3
Changed lines of the file:
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@@
 <?xml version="1.0" encoding="utf-8"?>
 <!DOCTYPE eagle SYSTEM "eagle.dtd">
-<eagle version="6.2">
+<eagle version="7.2.0">
 <drawing>
 <settings>
@@
 <part name="R1" library="SparkFun" deviceset="RESISTOR" device="0402-RES" value="DNP"/>
 <part name="R2" library="SparkFun" deviceset="RESISTOR" device="0402-RES" value="DNP"/>
-<part name="JP1" library="harwin" deviceset="M80-879" device="" value=""/>
+<part name="J1" library="harwin" deviceset="M80-879" device="" value=""/>
 <part name="SUPPLY1" library="supply2" deviceset="GND" device=""/>
 <part name="SUPPLY2" library="supply2" deviceset="GND" device=""/>
@@
 <instance part="R1" gate="G$1" x="134.62" y="116.84" rot="R90"/>
 <instance part="R2" gate="G$1" x="142.24" y="116.84" rot="R90"/>
-<instance part="JP1" gate="G$1" x="40.64" y="114.3"/>
+<instance part="J1" gate="G$1" x="40.64" y="114.3"/>
 <instance part="SUPPLY1" gate="GND" x="68.58" y="119.38"/>
 <instance part="SUPPLY2" gate="GND" x="83.82" y="88.9"/>
@@
 </busses>
 <nets>
-<net name="VCC" class="0">
+<net name="+3V3" class="0">
 <segment>
 <wire x1="127" y1="114.3" x2="129.54" y2="114.3" width="0.1524" layer="91"/>
@@
 <wire x1="53.34" y1="116.84" x2="63.5" y2="116.84" width="0.1524" layer="91"/>
 <label x="58.42" y="116.84" size="1.778" layer="95"/>
-<pinref part="JP1" gate="G$1" pin="2"/>
-</segment>
-</net>
-<net name="SCL" class="0">
+<pinref part="J1" gate="G$1" pin="2"/>
+</segment>
+</net>
+<net name="Q6_I2C_SCL_1" class="0">
 <segment>
 <wire x1="127" y1="109.22" x2="134.62" y2="109.22" width="0.1524" layer="91"/>
@@
 <wire x1="53.34" y1="106.68" x2="63.5" y2="106.68" width="0.1524" layer="91"/>
 <label x="58.42" y="106.68" size="1.778" layer="95"/>
-<pinref part="JP1" gate="G$1" pin="4"/>
-</segment>
-</net>
-<net name="SDA" class="0">
+<pinref part="J1" gate="G$1" pin="4"/>
+</segment>
+</net>
+<net name="Q6_I2C_SDA_1" class="0">
 <segment>
 <wire x1="127" y1="106.68" x2="142.24" y2="106.68" width="0.1524" layer="91"/>
@@
 <wire x1="53.34" y1="111.76" x2="63.5" y2="111.76" width="0.1524" layer="91"/>
 <label x="58.42" y="111.76" size="1.778" layer="95"/>
-<pinref part="JP1" gate="G$1" pin="3"/>
+<pinref part="J1" gate="G$1" pin="3"/>
 </segment>
 </net>
@@
 <wire x1="53.34" y1="121.92" x2="68.58" y2="121.92" width="0.1524" layer="91"/>
 <label x="58.42" y="121.92" size="1.778" layer="95"/>
-<pinref part="JP1" gate="G$1" pin="1"/>
+<pinref part="J1" gate="G$1" pin="1"/>
 <pinref part="SUPPLY1" gate="GND" pin="GND"/>
 </segment>
