File: CDH-V3.7/CDH-v3.7.brd (EAGLE design)
At the start: 90.6 x 91.8 mm, 47 parts, among them J2 M80-5000000M1-10-331-000, J3 M80-5000000M1-10-331-00-000, J4 SMFC

Commit message: Fixed all the trivial wiring issues for the CDH, Diplexer, EPS and wiring harness schematics
Connections:
- net ~PA3_JAG_TRST renamed ~PA3_JTAG_TRST
- removed net EXTERNAL_POWER_+V: H2.51, J3.X4
- removed net SLR_PNL_GND: H1.30
- new net EXTERNAL_POWER_V+: H2.52, J3.X3
- net EXTERNAL_POWER_GND: now also H2.51, J3.X4; no longer H2.52, J3.X3
- net SOLAR_PANEL_GND: now also H1.30
Routing:
- net EXTERNAL_POWER_V+: track 0.00 -> 25.3 mm
- net EXTERNAL_POWER_+V: track 18.2 -> 0.00 mm
- net EXTERNAL_POWER_GND: track 25.3 -> 18.2 mm
Changed lines of the file:
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@@
 <?xml version="1.0" encoding="utf-8"?>
 <!DOCTYPE eagle SYSTEM "eagle.dtd">
-<eagle version="7.2.0">
+<eagle version="7.3.0">
 <drawing>
 <settings>
@@
 <contactref element="J4" pad="29"/>
 </signal>
-<signal name="~PA3_JAG_TRST">
+<signal name="~PA3_JTAG_TRST">
 <contactref element="J4" pad="34"/>
 </signal>
@@
 <signal name="SOLAR_PANEL_GND">
 <contactref element="H1" pad="31"/>
+<contactref element="H1" pad="30"/>
+<wire x1="49.92203125" y1="83.963009375" x2="52.46203125" y2="81.423009375" width="0" layer="19" extent="1-1"/>
 </signal>
 <signal name="N$15">
@@
 <contactref element="U$6" pad="5"/>
 </signal>
-<signal name="EXTERNAL_POWER_+V">
+<signal name="EXTERNAL_POWER_GND">
 <contactref element="H2" pad="51"/>
 <contactref element="J3" pad="X4"/>
@@
 <via x="5.2832" y="3.175" extent="1-16" drill="3.2"/>
 </signal>
-<signal name="EXTERNAL_POWER_GND">
+<signal name="EXTERNAL_POWER_V+">
 <contactref element="H2" pad="52"/>
 <contactref element="J3" pad="X3"/>
@@
 <wire x1="84.05" y1="80.43" x2="84.05" y2="70.55" width="1.27" layer="1"/>
 </signal>
-<signal name="SLR_PNL_GND">
-<contactref element="H1" pad="30"/>
-</signal>
 <signal name="POW_9V">

Commit message: [CDH] updated trivial mismatches between connector netnames [EPS] updated trivial mismatches between connector netnames [PAYLOAD] updated trivial mismatches between connector netnames [WIRING] updated trivial mismatches between connector netnames
Connections:
- net BATTERY_THRMSTOR_+V renamed BATTERY_THRMSTOR1_+V
- net POW_RADIO_3.3V renamed POW_RADIO_3V3
- net POW_RADIO_3.3VSYS renamed POW_RADIO_3V3_SYS
- removed net N$84: H1.50
- net Q6_GPIO_10: now also H1.50
Changed lines of the file:
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@@
 <wire x1="78.2134" y1="53.775" x2="76.9112" y2="55.1222" width="0.8128" layer="16"/>
 </signal>
-<signal name="POW_RADIO_3.3VSYS">
+<signal name="POW_RADIO_3V3_SYS">
 <contactref element="H2" pad="28"/>
 </signal>
@@
 <wire x1="71.99" y1="59.83" x2="74.165" y2="61.1" width="0.4064" layer="16"/>
 </signal>
-<signal name="POW_RADIO_3.3V">
+<signal name="POW_RADIO_3V3">
 <contactref element="H2" pad="27"/>
 </signal>
@@
 <wire x1="50.74" y1="80.005" x2="51.15" y2="80.415" width="0.4064" layer="1"/>
 <wire x1="51.15" y1="80.415" x2="51.15" y2="82.650978125" width="0.4064" layer="1"/>
+<contactref element="H1" pad="50"/>
+<wire x1="52.46203125" y1="83.963009375" x2="75.32203125" y2="83.963009375" width="0" layer="19" extent="1-1"/>
 </signal>
 <signal name="Q6_GPIO_2">
@@
 <wire x1="18.2" y1="58.545" x2="18.635" y2="58.11" width="0.8128" layer="1"/>
 </signal>
-<signal name="BATTERY_THRMSTOR_+V">
+<signal name="BATTERY_THRMSTOR1_+V">
 <contactref element="H1" pad="8"/>
 <contactref element="J2" pad="X8"/>
@@
 <contactref element="H2" pad="48"/>
 </signal>
-<signal name="N$84">
-<contactref element="H1" pad="50"/>
-</signal>
 <signal name="THERMALGND1">

Commit message: Revert "Fixed all the trivial wiring issues for the CDH, Diplexer, EPS and wiring harness schematics"
This reverts commits
  6713d85a6277b26f983fd7a52d0f95a7f9e4e046.
  086194ae58682b6763f31692a26cd4dac33df983
  82b42737f0fe6cd82dfea4a4ae7507beb01cc7b8

This revert is required because changing/connecting net names in eagle will automatically modify or destroy PCB traces associated with those netnames.
Updating the schematics and PCBs will need to be redone carefully to ensure no traces are destroyed.

	modified:   CDH-V3.7/CDH-v3.7.brd
	modified:   CDH-V3.7/CDH-v3.7.sch
	modified:   Diplexer/diplexer_v4rev0-schematic.sch
	modified:   EPS/eps-v1-0.brd
	modified:   EPS/eps-v1-0.sch
	modified:   Payload Internal - Auxiliary/Payload v2.1.brd
	modified:   Payload Internal - Auxiliary/Payload v2.1.sch
	modified:   Wiring Harness/wiring-harness-complete-v1.0.sch
Connections:
- net BATTERY_THRMSTOR1_+V renamed BATTERY_THRMSTOR_+V
- net POW_RADIO_3V3 renamed POW_RADIO_3.3V
- net POW_RADIO_3V3_SYS renamed POW_RADIO_3.3VSYS
- net ~PA3_JTAG_TRST renamed ~PA3_JAG_TRST
- removed net EXTERNAL_POWER_V+: H2.52, J3.X3
- new net EXTERNAL_POWER_+V: H2.51, J3.X4
- new net N$84: H1.50
- new net SLR_PNL_GND: H1.30
- net EXTERNAL_POWER_GND: now also H2.52, J3.X3; no longer H2.51, J3.X4
- net Q6_GPIO_10: no longer H1.50
- net SOLAR_PANEL_GND: no longer H1.30
Routing:
- net EXTERNAL_POWER_V+: track 25.3 -> 0.00 mm
- net EXTERNAL_POWER_+V: track 0.00 -> 18.2 mm
- net EXTERNAL_POWER_GND: track 18.2 -> 25.3 mm
Changed lines of the file:
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@@
 <?xml version="1.0" encoding="utf-8"?>
 <!DOCTYPE eagle SYSTEM "eagle.dtd">
-<eagle version="7.3.0">
+<eagle version="7.2.0">
 <drawing>
 <settings>
@@
 <wire x1="78.2134" y1="53.775" x2="76.9112" y2="55.1222" width="0.8128" layer="16"/>
 </signal>
-<signal name="POW_RADIO_3V3_SYS">
+<signal name="POW_RADIO_3.3VSYS">
 <contactref element="H2" pad="28"/>
 </signal>
@@
 <wire x1="71.99" y1="59.83" x2="74.165" y2="61.1" width="0.4064" layer="16"/>
 </signal>
-<signal name="POW_RADIO_3V3">
+<signal name="POW_RADIO_3.3V">
 <contactref element="H2" pad="27"/>
 </signal>
@@
 <wire x1="50.74" y1="80.005" x2="51.15" y2="80.415" width="0.4064" layer="1"/>
 <wire x1="51.15" y1="80.415" x2="51.15" y2="82.650978125" width="0.4064" layer="1"/>
-<contactref element="H1" pad="50"/>
-<wire x1="52.46203125" y1="83.963009375" x2="75.32203125" y2="83.963009375" width="0" layer="19" extent="1-1"/>
 </signal>
 <signal name="Q6_GPIO_2">
@@
 <contactref element="J4" pad="29"/>
 </signal>
-<signal name="~PA3_JTAG_TRST">
+<signal name="~PA3_JAG_TRST">
 <contactref element="J4" pad="34"/>
 </signal>
@@
 <wire x1="18.2" y1="58.545" x2="18.635" y2="58.11" width="0.8128" layer="1"/>
 </signal>
-<signal name="BATTERY_THRMSTOR1_+V">
+<signal name="BATTERY_THRMSTOR_+V">
 <contactref element="H1" pad="8"/>
 <contactref element="J2" pad="X8"/>
@@
 <signal name="SOLAR_PANEL_GND">
 <contactref element="H1" pad="31"/>
-<contactref element="H1" pad="30"/>
-<wire x1="49.92203125" y1="83.963009375" x2="52.46203125" y2="81.423009375" width="0" layer="19" extent="1-1"/>
 </signal>
 <signal name="N$15">
@@
 <contactref element="U$6" pad="5"/>
 </signal>
-<signal name="EXTERNAL_POWER_GND">
+<signal name="EXTERNAL_POWER_+V">
 <contactref element="H2" pad="51"/>
 <contactref element="J3" pad="X4"/>
@@
 <contactref element="H2" pad="48"/>
 </signal>
+<signal name="N$84">
+<contactref element="H1" pad="50"/>
+</signal>
 <signal name="THERMALGND1">
 <contactref element="H1" pad="5"/>
@@
 <via x="5.2832" y="3.175" extent="1-16" drill="3.2"/>
 </signal>
-<signal name="EXTERNAL_POWER_V+">
+<signal name="EXTERNAL_POWER_GND">
 <contactref element="H2" pad="52"/>
 <contactref element="J3" pad="X3"/>
@@
 <wire x1="84.05" y1="80.43" x2="84.05" y2="70.55" width="1.27" layer="1"/>
 </signal>
+<signal name="SLR_PNL_GND">
+<contactref element="H1" pad="30"/>
+</signal>
 <signal name="POW_9V">
