File: CDH-V3.7/CDH-v3.7.sch (EAGLE design)
At the start: 47 parts

Commit message: CDH updates   - renamed H1 <-> H2 headers to match others schematics   - deleted misleading 'Q6_GPIO_10' label
Wiring harness updates
  - deleted misleading 'Q6_GPIO_10' label
Connections:
- net +3V3: now also H2.36, H2.38; no longer H1.36, H1.38
- net ANTENNA_DEPLOYMENT_+V: now also H1.1; no longer H2.1
- net ANTENNA_DEPLOYMENT_GND: now also H1.3; no longer H2.3
- net BATTERY_HEATER_+V: now also H1.4; no longer H2.4
- net BATTERY_HEATER_-V: now also H1.6; no longer H2.6
- net BATTERY_THRMSTOR2_+V: now also H1.12; no longer H2.12
- net BATTERY_THRMSTOR_+V: now also H1.8; no longer H2.8
- net BATTERY_THRMSTOR_-V: now also H1.10; no longer H2.10
- net BOTTOM_TEMP_SOLAR_PANEL-1: now also H2.9; no longer H1.9
- net BOTTOM_TEMP_SOLAR_PANEL-2: now also H2.11; no longer H1.11
- net BOTTOM_TEMP_SOLAR_PANEL-3: now also H2.13; no longer H1.13
- net BOTTOM_TEMP_SOLAR_PANEL-4: now also H2.15; no longer H1.15
- net ELEC_BAY_TEMP_1: now also H2.50; no longer H1.50
- net EXTERNAL_POWER_+V: now also H2.51; no longer H1.51
- net EXTERNAL_POWER_GND: now also H2.52; no longer H1.52
- net GND: now also H1.15, H1.23, H1.27, H1.34, H1.37, H1.41, H1.44, H1.45, H1.48, H1.49, H1.52, H2.16, H2.17, H2.22, H2.26, H2.4; no longer H1.16, H1.17, H1.22, H1.26, H1.4, H2.15, H2.23, H2.27, H2.34, H2.37, H2.41, H2.44, H2.45, H2.48, H2.49, H2.52
- net MECH_DEPLOY_SWITCH_+V: now also H2.31; no longer H1.31
- net MECH_DEPLOY_SWITCH_-V: now also H2.33; no longer H1.33
- net N$1: now also H2.6; no longer H1.6
- net N$11: now also H2.2; no longer H1.2
- net N$13: now also H2.49; no longer H1.49
- net N$15: now also H2.47; no longer H1.47
- net N$22: now also H2.34; no longer H1.34
- net N$27: now also H2.44; no longer H1.44
- net N$4: now also H2.8; no longer H1.8
- net N$5: now also H2.48; no longer H1.48
- net N$6: now also H2.10; no longer H1.10
- net N$78: now also H2.39; no longer H1.39
- net N$79: now also H2.41; no longer H1.41
- net N$80: now also H2.43; no longer H1.43
- net N$81: now also H2.40; no longer H1.40
- net N$83: now also H1.46; no longer H2.46
- net N$84: now also H1.50; no longer H2.50
- net N$9: now also H2.12; no longer H1.12
- net PC_Q6_RS232: now also H1.21; no longer H2.21
- net POW_3V3: now also H1.16, H1.20; no longer H2.16, H2.20
- net POW_5V: now also H1.26, H1.28; no longer H2.26, H2.28
- net POW_9V: now also H1.22, H1.24; no longer H2.22, H2.24
- net POW_BATT_GND: now also H1.33; no longer H2.33
- net POW_BATT_VOUT: now also H1.35; no longer H2.35
- net POW_RADIO_3.3V: now also H2.27; no longer H1.27
- net POW_RADIO_3.3VSYS: now also H2.28; no longer H1.28
- net POW_RADIO_GND: now also H2.29, H2.30, H2.32; no longer H1.29, H1.30, H1.32
- net POW_RADIO_VBATT: now also H2.45, H2.46; no longer H1.45, H1.46
- net Q6_AIN_0: now also H1.39; no longer H2.39
- net Q6_AIN_1: now also H1.43; no longer H2.43
- net Q6_AOUT_0: now also H1.47; no longer H2.47
- net Q6_AOUT_1: now also H1.51; no longer H2.51
- net Q6_GPIO_0: now also H1.13; no longer H2.13
- net Q6_GPIO_10: now also H1.32; no longer H2.32
- net Q6_GPIO_13: now also H1.36; no longer H2.36
- net Q6_GPIO_14: now also H1.38; no longer H2.38
- net Q6_GPIO_15: now also H1.40; no longer H2.40
- net Q6_GPIO_2: now also H2.24; no longer H1.24
- net Q6_GPIO_6: now also H1.7; no longer H2.7
- net Q6_GPIO_7: now also H1.9; no longer H2.9
- net Q6_GPIO_8: now also H1.11; no longer H2.11
- net Q6_I2C_SCL_1: now also H2.20; no longer H1.20
- net Q6_I2C_SDA_1: now also H2.18; no longer H1.18
- net Q6_PC_RS232: now also H1.25; no longer H2.25
- net Q6_RADIO_UART_RX: now also H1.18; no longer H2.18
- net Q6_RADIO_UART_TX: now also H1.17; no longer H2.17
- net Q6_SPI_CS0: now also H2.37; no longer H1.37
- net Q6_SPI_CS1: now also H2.25; no longer H1.25
- net Q6_SPI_SCLK: now also H2.21; no longer H1.21
- net Q6_SPI_SDI_MISO: now also H2.35; no longer H1.35
- net Q6_SPI_SDO_MOSI: now also H2.23; no longer H1.23
- net SLR_PNL_GND: now also H1.30; no longer H2.30
- net SOLAR_PANEL_1_3: now also H1.29; no longer H2.29
- net SOLAR_PANEL_2_4: now also H1.2; no longer H2.2
- net SOLAR_PANEL_GND: now also H1.31; no longer H2.31
- net THERMALGND1: now also H1.5; no longer H2.5
- net TOP_TEMP_SOLAR_PANEL-1: now also H2.1; no longer H1.1
- net TOP_TEMP_SOLAR_PANEL-2: now also H2.3; no longer H1.3
- net TOP_TEMP_SOLAR_PANEL-3: now also H2.5; no longer H1.5
- net TOP_TEMP_SOLAR_PANEL-4: now also H2.7; no longer H1.7
Other:
- note removed: "Q6_GPIO_10"
- moved on the sheet: H1, H2

Commit message: [CDH] renamed connectors to 'J#' in sync with wiring harness [diplexer-rcl.lbr] copied rcl.lbr and created an inductor with SMD package L01005(imperial) [DIPLEXER] renamed sma connectors to 'J#' in sync with wiring harness    changed part symbols of C6 C7 C8 C9 C10 to L6 L7 L8 L9 L10 [space-concordia-power-lbr] updated 'GLENAIR-171-006-6-S-6-7-18' to have a valid prefix [Payload-Internal-Aux] renamed connectors to 'J#' in sync with wiring harness [wiring-harness] renamed all known connectors to 'J#' in sync with wiring harness
Parts:
- renumbered U$1 to J4, U$2 to J2, U$3 to J3

Commit message: Fixed all the trivial wiring issues for the CDH, Diplexer, EPS and wiring harness schematics
Connections:
- net ~PA3_JAG_TRST renamed ~PA3_JTAG_TRST
- removed net EXTERNAL_POWER_+V: H2.51, J3.X4
- removed net SLR_PNL_GND: H1.30
- new net EXTERNAL_POWER_V+: H2.52, J3.X3
- net EXTERNAL_POWER_GND: now also H2.51, J3.X4; no longer H2.52, J3.X3
- net SOLAR_PANEL_GND: now also H1.30
Changed lines of the file:
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@@
 <?xml version="1.0" encoding="utf-8"?>
 <!DOCTYPE eagle SYSTEM "eagle.dtd">
-<eagle version="7.2.0">
+<eagle version="7.3.0">
 <drawing>
 <settings>
@@
 </segment>
 </net>
-<net name="~PA3_JAG_TRST" class="0">
+<net name="~PA3_JTAG_TRST" class="0">
 <segment>
 <pinref part="J4" gate="G$1" pin="C34"/>
@@
 <label x="-139.7" y="-68.58" size="1.778" layer="95"/>
 </segment>
+<segment>
+<pinref part="H1" gate="G$1" pin="30"/>
+<wire x1="-91.44" y1="-66.04" x2="-53.34" y2="-66.04" width="0.1524" layer="91"/>
+<label x="-81.28" y="-66.04" size="1.778" layer="95"/>
+</segment>
 </net>
 <net name="N$15" class="0">
@@
 </segment>
 </net>
-<net name="EXTERNAL_POWER_+V" class="0">
+<net name="EXTERNAL_POWER_GND" class="0">
 <segment>
 <pinref part="H2" gate="G$1" pin="51"/>
@@
 </segment>
 </net>
-<net name="EXTERNAL_POWER_GND" class="0">
+<net name="EXTERNAL_POWER_V+" class="0">
 <segment>
 <pinref part="H2" gate="G$1" pin="52"/>
@@
 </segment>
 </net>
-<net name="SLR_PNL_GND" class="0">
-<segment>
-<pinref part="H1" gate="G$1" pin="30"/>
-<wire x1="-91.44" y1="-66.04" x2="-53.34" y2="-66.04" width="0.1524" layer="91"/>
-<label x="-81.28" y="-66.04" size="1.778" layer="95"/>
-</segment>
-</net>

Commit message: [CDH] updated trivial mismatches between connector netnames [EPS] updated trivial mismatches between connector netnames [PAYLOAD] updated trivial mismatches between connector netnames [WIRING] updated trivial mismatches between connector netnames
Connections:
- net BATTERY_THRMSTOR_+V renamed BATTERY_THRMSTOR1_+V
- net POW_RADIO_3.3V renamed POW_RADIO_3V3
- net POW_RADIO_3.3VSYS renamed POW_RADIO_3V3_SYS
- removed net N$84: H1.50
- net Q6_GPIO_10: now also H1.50
Changed lines of the file:
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@@
 </segment>
 </net>
-<net name="POW_RADIO_3.3VSYS" class="0">
+<net name="POW_RADIO_3V3_SYS" class="0">
 <segment>
 <pinref part="H2" gate="G$1" pin="28"/>
@@
 </segment>
 </net>
-<net name="POW_RADIO_3.3V" class="0">
+<net name="POW_RADIO_3V3" class="0">
 <segment>
 <pinref part="H2" gate="G$1" pin="27"/>
@@
 <wire x1="-91.44" y1="-68.58" x2="-53.34" y2="-68.58" width="0.1524" layer="91"/>
 <label x="-81.28" y="-68.58" size="1.778" layer="95"/>
+</segment>
+<segment>
+<pinref part="H1" gate="G$1" pin="50"/>
+<wire x1="-91.44" y1="-91.44" x2="-52.07" y2="-91.44" width="0.1524" layer="91"/>
+<label x="-81.28" y="-91.44" size="1.778" layer="95"/>
 </segment>
 </net>
@@
 </segment>
 </net>
-<net name="BATTERY_THRMSTOR_+V" class="0">
+<net name="BATTERY_THRMSTOR1_+V" class="0">
 <segment>
 <pinref part="H1" gate="G$1" pin="8"/>
@@
 </segment>
 </net>
-<net name="N$84" class="0">
-<segment>
-<pinref part="H1" gate="G$1" pin="50"/>
-<wire x1="-91.44" y1="-91.44" x2="-52.07" y2="-91.44" width="0.1524" layer="91"/>
-<label x="-81.28" y="-91.44" size="1.778" layer="95"/>
-</segment>
-</net>

Commit message: Revert "Fixed all the trivial wiring issues for the CDH, Diplexer, EPS and wiring harness schematics"
This reverts commits
  6713d85a6277b26f983fd7a52d0f95a7f9e4e046.
  086194ae58682b6763f31692a26cd4dac33df983
  82b42737f0fe6cd82dfea4a4ae7507beb01cc7b8

This revert is required because changing/connecting net names in eagle will automatically modify or destroy PCB traces associated with those netnames.
Updating the schematics and PCBs will need to be redone carefully to ensure no traces are destroyed.

	modified:   CDH-V3.7/CDH-v3.7.brd
	modified:   CDH-V3.7/CDH-v3.7.sch
	modified:   Diplexer/diplexer_v4rev0-schematic.sch
	modified:   EPS/eps-v1-0.brd
	modified:   EPS/eps-v1-0.sch
	modified:   Payload Internal - Auxiliary/Payload v2.1.brd
	modified:   Payload Internal - Auxiliary/Payload v2.1.sch
	modified:   Wiring Harness/wiring-harness-complete-v1.0.sch
Connections:
- net BATTERY_THRMSTOR1_+V renamed BATTERY_THRMSTOR_+V
- net POW_RADIO_3V3 renamed POW_RADIO_3.3V
- net POW_RADIO_3V3_SYS renamed POW_RADIO_3.3VSYS
- net ~PA3_JTAG_TRST renamed ~PA3_JAG_TRST
- removed net EXTERNAL_POWER_V+: H2.52, J3.X3
- new net EXTERNAL_POWER_+V: H2.51, J3.X4
- new net N$84: H1.50
- new net SLR_PNL_GND: H1.30
- net EXTERNAL_POWER_GND: now also H2.52, J3.X3; no longer H2.51, J3.X4
- net Q6_GPIO_10: no longer H1.50
- net SOLAR_PANEL_GND: no longer H1.30
Changed lines of the file:
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@@
 <?xml version="1.0" encoding="utf-8"?>
 <!DOCTYPE eagle SYSTEM "eagle.dtd">
-<eagle version="7.3.0">
+<eagle version="7.2.0">
 <drawing>
 <settings>
@@
 </segment>
 </net>
-<net name="POW_RADIO_3V3_SYS" class="0">
+<net name="POW_RADIO_3.3VSYS" class="0">
 <segment>
 <pinref part="H2" gate="G$1" pin="28"/>
@@
 </segment>
 </net>
-<net name="POW_RADIO_3V3" class="0">
+<net name="POW_RADIO_3.3V" class="0">
 <segment>
 <pinref part="H2" gate="G$1" pin="27"/>
@@
 <wire x1="-91.44" y1="-68.58" x2="-53.34" y2="-68.58" width="0.1524" layer="91"/>
 <label x="-81.28" y="-68.58" size="1.778" layer="95"/>
-</segment>
-<segment>
-<pinref part="H1" gate="G$1" pin="50"/>
-<wire x1="-91.44" y1="-91.44" x2="-52.07" y2="-91.44" width="0.1524" layer="91"/>
-<label x="-81.28" y="-91.44" size="1.778" layer="95"/>
 </segment>
 </net>
@@
 </segment>
 </net>
-<net name="~PA3_JTAG_TRST" class="0">
+<net name="~PA3_JAG_TRST" class="0">
 <segment>
 <pinref part="J4" gate="G$1" pin="C34"/>
@@
 </segment>
 </net>
-<net name="BATTERY_THRMSTOR1_+V" class="0">
+<net name="BATTERY_THRMSTOR_+V" class="0">
 <segment>
 <pinref part="H1" gate="G$1" pin="8"/>
@@
 <label x="-139.7" y="-68.58" size="1.778" layer="95"/>
 </segment>
-<segment>
-<pinref part="H1" gate="G$1" pin="30"/>
-<wire x1="-91.44" y1="-66.04" x2="-53.34" y2="-66.04" width="0.1524" layer="91"/>
-<label x="-81.28" y="-66.04" size="1.778" layer="95"/>
-</segment>
 </net>
 <net name="N$15" class="0">
@@
 </segment>
 </net>
-<net name="EXTERNAL_POWER_GND" class="0">
+<net name="EXTERNAL_POWER_+V" class="0">
 <segment>
 <pinref part="H2" gate="G$1" pin="51"/>
@@
 <wire x1="-91.44" y1="-10.16" x2="-55.88" y2="-10.16" width="0.1524" layer="91"/>
 <label x="-63.5" y="-10.16" size="1.778" layer="95"/>
+</segment>
+</net>
+<net name="N$84" class="0">
+<segment>
+<pinref part="H1" gate="G$1" pin="50"/>
+<wire x1="-91.44" y1="-91.44" x2="-52.07" y2="-91.44" width="0.1524" layer="91"/>
+<label x="-81.28" y="-91.44" size="1.778" layer="95"/>
 </segment>
 </net>
@@
 </segment>
 </net>
-<net name="EXTERNAL_POWER_V+" class="0">
+<net name="EXTERNAL_POWER_GND" class="0">
 <segment>
 <pinref part="H2" gate="G$1" pin="52"/>
@@
 </segment>
 </net>
+<net name="SLR_PNL_GND" class="0">
+<segment>
+<pinref part="H1" gate="G$1" pin="30"/>
+<wire x1="-91.44" y1="-66.04" x2="-53.34" y2="-66.04" width="0.1524" layer="91"/>
+<label x="-81.28" y="-66.04" size="1.778" layer="95"/>
+</segment>
+</net>

Commit message: [CDH] - fixed typos in signal netnames so they match wiring-harness   - updated 'EXTERNAL_POWER_+V' and 'EXTERNAL_POWER_GND' so that they match the EPS header [WIRING] - updated 'EXTERNAL_POWER_+V' and 'EXTERNAL_POWER_GND' so that they properly route through the wiring harness
Connections:
- net ~PA3_JAG_TRST renamed ~PA3_JTAG_TRST
- net EXTERNAL_POWER_+V: now also H2.52, J3.X3; no longer H2.51, J3.X4
- net EXTERNAL_POWER_GND: now also H2.51, J3.X4; no longer H2.52, J3.X3
Changed lines of the file:
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@@
 <?xml version="1.0" encoding="utf-8"?>
 <!DOCTYPE eagle SYSTEM "eagle.dtd">
-<eagle version="7.2.0">
+<eagle version="7.3.0">
 <drawing>
 <settings>
@@
 </segment>
 </net>
-<net name="~PA3_JAG_TRST" class="0">
+<net name="~PA3_JTAG_TRST" class="0">
 <segment>
 <pinref part="J4" gate="G$1" pin="C34"/>
@@
 </segment>
 </net>
-<net name="EXTERNAL_POWER_+V" class="0">
+<net name="EXTERNAL_POWER_GND" class="0">
 <segment>
 <pinref part="H2" gate="G$1" pin="51"/>
@@
 </segment>
 </net>
-<net name="EXTERNAL_POWER_GND" class="0">
+<net name="EXTERNAL_POWER_+V" class="0">
 <segment>
 <pinref part="H2" gate="G$1" pin="52"/>

Commit message: [CDH] [Wiring Harness] [Payload-Internal-Aux] renamed nets 'Q6_PC_RS232' and 'PC_Q6_RS232' to 'Q6_MAX_RS232' and 'MAX_Q6_RS232' for clarity
Connections:
- net PC_Q6_RS232 renamed MAX_Q6_RS232
- net Q6_PC_RS232 renamed Q6_MAX_RS232
- removed net SLR_PNL_GND: H1.30
- net SOLAR_PANEL_GND: now also H1.30
Changed lines of the file:
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@@
 </segment>
 </net>
-<net name="PC_Q6_RS232" class="0">
+<net name="MAX_Q6_RS232" class="0">
 <segment>
 <pinref part="J4" gate="G$1" pin="C44"/>
@@
 </segment>
 </net>
-<net name="Q6_PC_RS232" class="0">
+<net name="Q6_MAX_RS232" class="0">
 <segment>
 <pinref part="J4" gate="G$1" pin="C42"/>
@@
 <wire x1="-114.3" y1="-68.58" x2="-142.24" y2="-68.58" width="0.1524" layer="91"/>
 <label x="-139.7" y="-68.58" size="1.778" layer="95"/>
+</segment>
+<segment>
+<pinref part="H1" gate="G$1" pin="30"/>
+<wire x1="-91.44" y1="-66.04" x2="-53.34" y2="-66.04" width="0.1524" layer="91"/>
+<label x="-81.28" y="-66.04" size="1.778" layer="95"/>
 </segment>
 </net>
@@
 </segment>
 </net>
-<net name="SLR_PNL_GND" class="0">
-<segment>
-<pinref part="H1" gate="G$1" pin="30"/>
-<wire x1="-91.44" y1="-66.04" x2="-53.34" y2="-66.04" width="0.1524" layer="91"/>
-<label x="-81.28" y="-66.04" size="1.778" layer="95"/>
-</segment>
-</net>
