File: Diplexer/diplexer_v4rev0-schematic.sch (EAGLE design)
At the start: 13 parts, among them J10 SMA-142-0701-801/806, J11 SMA-142-0701-801/806, J12 SMA-142-0701-801/806

Commit message: Revert "Fixed all the trivial wiring issues for the CDH, Diplexer, EPS and wiring harness schematics"
This reverts commits
  6713d85a6277b26f983fd7a52d0f95a7f9e4e046.
  086194ae58682b6763f31692a26cd4dac33df983
  82b42737f0fe6cd82dfea4a4ae7507beb01cc7b8

This revert is required because changing/connecting net names in eagle will automatically modify or destroy PCB traces associated with those netnames.
Updating the schematics and PCBs will need to be redone carefully to ensure no traces are destroyed.

	modified:   CDH-V3.7/CDH-v3.7.brd
	modified:   CDH-V3.7/CDH-v3.7.sch
	modified:   Diplexer/diplexer_v4rev0-schematic.sch
	modified:   EPS/eps-v1-0.brd
	modified:   EPS/eps-v1-0.sch
	modified:   Payload Internal - Auxiliary/Payload v2.1.brd
	modified:   Payload Internal - Auxiliary/Payload v2.1.sch
	modified:   Wiring Harness/wiring-harness-complete-v1.0.sch
Connections:
- net DIPLEX_TO_ANT_SIG renamed N$6
- net HE100_RX_TO_DIPLEX_SIG renamed N$2
- net HE100_TX_TO_DIPLEX_SIG renamed N$5
Changed lines of the file:
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@@
 <?xml version="1.0" encoding="utf-8"?>
 <!DOCTYPE eagle SYSTEM "eagle.dtd">
-<eagle version="7.3.0">
+<eagle version="7.2.0">
 <drawing>
 <settings>
@@
 <setting verticaltext="up"/>
 </settings>
-<grid distance="0.1" unitdist="inch" unit="inch" style="lines" multiple="1" display="no" altdistance="0.01" altunitdist="inch" altunit="inch"/>
+<grid distance="0.05" unitdist="inch" unit="inch" style="lines" multiple="1" display="no" altdistance="0.01" altunitdist="inch" altunit="inch"/>
 <layers>
 <layer number="1" name="Top" color="4" fill="1" visible="no" active="no"/>
@@
 </segment>
 </net>
-<net name="HE100_TX_TO_DIPLEX_SIG" class="0">
+<net name="N$5" class="0">
 <segment>
 <pinref part="J11" gate="G1" pin="1"/>
@@
 </segment>
 </net>
-<net name="HE100_RX_TO_DIPLEX_SIG" class="0">
+<net name="N$2" class="0">
 <segment>
 <pinref part="J10" gate="G1" pin="1"/>
@@
 </segment>
 </net>
-<net name="DIPLEX_TO_ANT_SIG" class="0">
+<net name="N$6" class="0">
 <segment>
 <pinref part="C3" gate="G$1" pin="2"/>

Commit message: [DIPLEXER] - updated netnames to match wiring harness netnames [WIRING] - updated parts J10,J11 and J12 to match the correct coax connector used on the diplexer
Connections:
- net N$2 renamed HE100_RX_TO_DIPLEX_SIG
- net N$5 renamed HE100_TX_TO_DIPLEX_SIG
- net N$6 renamed DIPLEX_TO_ANT_SIG
Changed lines of the file:
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@@
 <?xml version="1.0" encoding="utf-8"?>
 <!DOCTYPE eagle SYSTEM "eagle.dtd">
-<eagle version="7.2.0">
+<eagle version="7.3.0">
 <drawing>
 <settings>
@@
 <setting verticaltext="up"/>
 </settings>
-<grid distance="0.05" unitdist="inch" unit="inch" style="lines" multiple="1" display="no" altdistance="0.01" altunitdist="inch" altunit="inch"/>
+<grid distance="0.1" unitdist="inch" unit="inch" style="lines" multiple="1" display="no" altdistance="0.01" altunitdist="inch" altunit="inch"/>
 <layers>
 <layer number="1" name="Top" color="4" fill="1" visible="no" active="no"/>
@@
 </segment>
 </net>
-<net name="N$5" class="0">
+<net name="HE100_TX_TO_DIPLEX_SIG" class="0">
 <segment>
 <pinref part="J11" gate="G1" pin="1"/>
@@
 </segment>
 </net>
-<net name="N$2" class="0">
+<net name="HE100_RX_TO_DIPLEX_SIG" class="0">
 <segment>
 <pinref part="J10" gate="G1" pin="1"/>
@@
 </segment>
 </net>
-<net name="N$6" class="0">
+<net name="DIPLEX_TO_ANT_SIG" class="0">
 <segment>
 <pinref part="C3" gate="G$1" pin="2"/>
